Commit message: doulevei to PD olee

File: src/cepheus_description/urdf/simple_ring.xacro (robot description, xacro)
@@ -3,4 +3,96 @@
   <xacro:include filename="$(find cepheus_description)/urdf/simple_ring.gazebo" />
   <link name="world"></link>
+	<!-- <joint name="p1_joint" type="prismatic">
+		<parent link="world"/>
+		<child link="p1"/>
+		<axis xyz="1 0 0"/>
+		<limit lower="-100" upper="100" effort="1000" velocity="10000"/>
+		<dynamics damping="0" friction="0"/>
+	</joint>
+	<link name="p1">
+		<inertial>
+			<origin
+				xyz="0.0 0.0 0.0"
+				rpy="0.0 0.0 0.0" />
+			<mass value="0.01" />
+			<inertia
+				ixx="1e-2"
+				ixy="0.0"
+				ixz="0.0"
+				iyy="1e-2"
+				iyz="0.0"
+				izz="1e-2" />
+		</inertial>
+	</link>
+	<gazebo reference="p1">
+		<mu1>0</mu1>
+		<mu2>0</mu2>
+	</gazebo>
+	<transmission name="lin1">
+		<type>transmission_interface/SimpleTransmission</type>
+		<joint name="p1_joint">
+			<hardwareInterface>hardware_interface/EffortJointInterface</hardwareInterface>
+		</joint>
+		<actuator name="lin_motor1">
+			<hardwareInterface>EffortJointInterface</hardwareInterface>
+			<mechanicalReduction>1</mechanicalReduction>
+		</actuator>
+	</transmission>
+	<joint name="p2_joint" type="prismatic">
+		<parent link="p1"/>
+		<child link="p2"/>
+		<axis xyz="0 1 0"/>
+		<limit
+			lower="-100"
+			upper="100"
+			effort="1000"
+			velocity="10000"/>
+		<dynamics
+			damping="0"
+			friction="0"/>
+	</joint>
+	<link name="p2">
+		<inertial>
+			<origin
+				xyz="0.0 0.0 0.0"
+				rpy="0.0 0.0 0.0" />
+			<mass value="0.01" />
+			<inertia
+				ixx="1e-2"
+				ixy="0.0"
+				ixz="0.0"
+				iyy="1e-2"
+				iyz="0.0"
+				izz="1e-2" />
+		</inertial>
+		<surface>
+			<friction>
+				<ode>
+					<mu>0</mu>
+					<mu2>0</mu2>
+					<fdir1>0 1.0 0</fdir1>
+					<implicit_spring_damper>true</implicit_spring_damper>
+				</ode>
+			</friction>
+		</surface>
+	</link>
+	<gazebo reference="p2">
+		<mu1>0</mu1>
+		<mu2>0</mu2>
+	</gazebo>
+	<transmission name="lin2">
+		<type>transmission_interface/SimpleTransmission</type>
+		<joint name="p2_joint">
+			<hardwareInterface>hardware_interface/EffortJointInterface</hardwareInterface>
+		</joint>
+		<actuator name="lin_motor2">
+			<hardwareInterface>EffortJointInterface</hardwareInterface>
+			<mechanicalReduction>1</mechanicalReduction>
+		</actuator>
+	</transmission>
+  <joint name="fixed_joint" type="fixed">
+    <parent link="p2"/>
+    <origin link="base_link"/>
+  </joint> -->
   <joint name="base_joint" type="planar">
     <origin xyz = "5 0 0" rpy="0 0 0"/>
@@ -24,8 +116,12 @@
     </collision>
     <inertial>
-      <mass value="9.0"/>
+      <mass value="1.0"/>
       <inertia ixx="0.00833" ixy="0" ixz="0" iyy="0.00833" iyz="0" izz="0.00833"/>
     </inertial>
   </link>
+  <gazebo reference="base_link">
+      <mu1>0</mu1>
+      <mu2>0</mu2>
+  </gazebo>
 <!--
   <link name="ring_link">
