Commit message: katalava to gazebo

File: src/cepheus_description/urdf/only_gripper.xacro (robot description, xacro)
@@ -29,12 +29,12 @@
 	<xacro:property name="arm_mass" value="0.2314" />
 	<xacro:property name="forearm_mass" value="0.1" />
-	<xacro:property name="gripper_mass" value="0.046" />
+	<xacro:property name="gripper_mass" value="4.6" />
 	<xacro:property name="base_inertia" value="1.06" />
 	<xacro:property name="arm_inertia" value="0.0026476" />
 	<xacro:property name="forearm_inertia" value="0.0011318" />
 	<!-- <xacro:property name="gripper_inertia" value="${9.61/100000}" /> -->
-	<xacro:property name="gripper_inertia" value="${2.73/100000}" />
-	<xacro:property name="joint_damping" value="0" />
-	<xacro:property name="joint_friction" value="0" />
+	<xacro:property name="gripper_inertia" value="${2.73/1000}" />
+	<xacro:property name="joint_damping" value="1" />
+	<xacro:property name="joint_friction" value="1" />
 	<xacro:property name="joint_limit" value="3.14" />
 	<xacro:property name="joint_velocity" value="100000" />
@@ -53,13 +53,5 @@
 		</joint> -->
 	</link>
-	<!-- extra links addition START -->
-	<!-- <joint name="world_joint" type="continuous">
-		<axis xyz="0 0 1"/>
-		<parent link="world"/>
-		<origin rpy="0 0 0" xyz="0 0 0"/>
-		<child link="cepheus"/>
-		<dynamics damping="0" friction="0"/>
-	</joint> -->
-	<joint name="p1_joint" type="prismatic">
+    	<joint name="p1_joint" type="prismatic">
 		<parent link="world"/>
 		<child link="p1"/>
@@ -149,9 +141,9 @@
 		</actuator>
 	</transmission>
-	<joint name="r_joint" type="continuous">
+	<joint name="left_wrist_joint" type="continuous">
 		<axis xyz="0 0 1"/>
 		<parent link="p2"/>
 		<origin rpy="0 0 0" xyz="0 0 0"/>
-		<child link="cepheus_base"/>
+		<child link="left_grip"/>
 		<dynamics damping="${joint_damping}" friction="${joint_friction}"/>
 	</joint>
@@ -159,5 +151,5 @@
 		<type>
 			transmission_interface/SimpleTransmission</type>
-		<joint name="r_joint">
+		<joint name="left_wrist_joint">
 			<hardwareInterface>hardware_interface/EffortJointInterface</hardwareInterface>
 		</joint>
@@ -167,221 +159,4 @@
 		</actuator>
 	</transmission>
-	<!-- extra links addition END -->
-	<link name="cepheus_base">
-		<!-- <xacro:inertial_cylinder mass="53" length="0.43" radius="0.2">
-			<origin xyz="0.0024 0.02937 0.15711" rpy="0 0 0 "/>
-		</xacro:inertial_cylinder> -->
-		<inertial>
-			<origin xyz="0.0024 0.02937 0.15711" rpy="0 0 0" />
-			<mass value="${base_mass}"/>
-			<inertia
-				ixx="0.000001"
-				ixy="0.000001"
-				ixz="0.000001"
-				iyy="0.000001"
-				iyz="0.000001"
-				izz="${base_inertia}" />
-		</inertial>
-		<visual>
-			<origin
-				xyz="0 0 0.215"
-				rpy="0 0 0" />
-			<geometry>
-				<!-- <mesh filename="package://cepheus_description/urdf/meshes/cepheus.STL" /> -->
-				<cylinder length="0.43" radius="${base_radius}"/>
-			</geometry>
-			<material name="LightGrey"/>
-		</visual>
-		<collision>
-			<origin
-				xyz="0 0 0.215"
-				rpy="0 0 0" />
-			<geometry>
-				<cylinder length="0.43" radius="${base_radius}"/>
-			</geometry>
-		</collision>
-	</link>
-	<!-- <joint name="reaction_wheel_joint" type="continuous">
-		<parent link="cepheus_base"/>
-		<child link="reaction_wheel"/>
-		<origin xyz="0 0 0.03815" rpy="0 0 0 "/>
-		<axis xyz="0 0 1" />
-		<dynamics damping="${joint_damping}" friction="${joint_friction}"/>
-	</joint> -->
-	<!-- <link name="reaction_wheel">
-		<visual>
-			<material name="silver">
-				<color rgba="0.5 0.5 0.5 1"/>
-			</material>
-			<geometry>
-				<mesh filename="package://cepheus_description/urdf/meshes/reaction_wheel.STL" />
-			</geometry>
-			<origin xyz="0 0 0" rpy="0 0 0"/>
-		</visual>
-		<inertial>
-			<origin xyz="0 0 0.025" rpy="0 0 0" />
-			<mass value="0.001"/>
-			<inertia
-				ixx="0.000001"
-				ixy="0.000001"
-				ixz="0.000001"
-				iyy="0.000001"
-				iyz="0.000001"
-				izz="0.00000197" />
-		</inertial>
-	</link> -->
-	<gazebo reference="cepheus_base">
-		<mu1>0</mu1>
-		<mu2>0</mu2>
-	</gazebo>
-	<!-- <transmission name="tran1">
-		<type>
-			transmission_interface/SimpleTransmission</type>
-		<joint name="reaction_wheel_joint">
-			<hardwareInterface>hardware_interface/EffortJointInterface</hardwareInterface>
-		</joint>
-		<actuator name="motor1">
-			<hardwareInterface>hardware_interface/EffortJointInterface</hardwareInterface>
-			<mechanicalReduction>1</mechanicalReduction>
-		</actuator>
-	</transmission> -->
-	<joint name="left_shoulder_joint" type="revolute">
-		<origin
-			xyz="0.1425 -0.08225 0.05875"
-			rpy="0 0 0" />
-		<parent link="cepheus_base" />
-		<child link="left_arm" />
-		<axis xyz="0 0 1" />
-		<limit
-			lower="${-joint_limit}"
-			upper="${joint_limit}"
-			effort="${joint_effort}"
-			velocity="${joint_velocity}" />
-		<dynamics
-			damping="${joint_damping}"
-			friction="${joint_friction}" />
-	</joint>
-	<link name="left_arm">
-		<inertial>
-			<origin
-				xyz="${arm_length/2} 0 0"
-				rpy="0 0 0" />
-			<mass value="${arm_mass}" />
-			<inertia
-				ixx="0.000001"
-				ixy="0.000001"
-				ixz="0.000001"
-				iyy="0.000001"
-				iyz="0.000001"
-				izz="${arm_inertia}" />
-		</inertial>
-		<visual>
-			<origin
-				xyz="${arm_length/2} 0 0"
-				rpy="0 0 0" />
-			<geometry>
-				<box size="${arm_length} 0.02 0.02" />
-			</geometry>
-			<material name="LightGrey"/>
-		</visual>
-		<collision>
-			<origin
-				xyz="${arm_length/2} 0.0 0"
-				rpy="0 0 0" />
-			<geometry>
-				<box size="${arm_length} 0.02 0.02"/>
-			</geometry>
-		</collision>
-		<!-- <xacro:inertial_box mass="0.2314" x="0.37" y="0.02" z="0.02">
-			<origin xyz="0.185 0 0" rpy="0 0 0"/>
-		</xacro:inertial_box> -->
-	</link>
-	<transmission name="tran2">
-		<type>transmission_interface/SimpleTransmission</type>
-		<joint name="left_shoulder_joint">
-			<hardwareInterface>hardware_interface/EffortJointInterface</hardwareInterface>
-		</joint>
-		<actuator name="motor2">
-			<hardwareInterface>hardware_interface/EffortJointInterface</hardwareInterface>
-			<mechanicalReduction>1</mechanicalReduction>
-		</actuator>
-	</transmission>
-	<joint name="left_elbow_joint" type="revolute">
-		<origin
-			xyz="${arm_length} 0 0"
-			rpy="0 0 0" />
-		<parent link="left_arm" />
-		<child link="left_forearm" />
-		<axis xyz="0 0 1" />
-		<limit
-			lower="${-joint_limit}"
-			upper="${joint_limit}"
-			effort="${joint_effort}"
-			velocity="${joint_velocity}" />
-		<dynamics
-			damping="${joint_damping}"
-			friction="${joint_friction}" />
-	</joint>
-	<link name="left_forearm">
-		<inertial>
-			<origin
-				xyz="${forearm_length/2} 0 0"
-				rpy="0 0 0" />
-			<mass value="${forearm_mass}" />
-			<inertia
-				ixx="0.000001"
-				ixy="0.000001"
-				ixz="0.000001"
-				iyy="0.000001"
-				iyz="0.000001"
-				izz="${forearm_inertia}" />
-		</inertial>
-		<visual>
-			<origin
-				xyz="${forearm_length/2} 0 0"
-				rpy="0 0 0" />
-			<geometry>
-				<box size="${forearm_length} 0.02 0.02"/>
-			</geometry>
-			<material name="LightGrey"/>
-		</visual>
-		<collision>
-			<origin
-				xyz="${forearm_length/2} 0 0"
-				rpy="0 0 0" />
-			<geometry>
-				<box size="${forearm_length} 0.02 0.02"/>
-			</geometry>
-		</collision>
-		<!-- <xacro:inertial_box mass="0.1" x="0.286" y="0.02" z="0.02">
-			<origin xyz="0.143 0 0" rpy="0 0 0"/>
-		</xacro:inertial_box> -->
-	</link>
-	<transmission name="tran3">
-		<type>transmission_interface/SimpleTransmission</type>
-		<joint name="left_elbow_joint">
-			<hardwareInterface>hardware_interface/EffortJointInterface</hardwareInterface>
-		</joint>
-		<actuator name="motor3">
-			<hardwareInterface>hardware_interface/EffortJointInterface</hardwareInterface>
-			<mechanicalReduction>1</mechanicalReduction>
-		</actuator>
-	</transmission>
-	<joint name="left_wrist_joint" type="revolute">
-		<origin
-			xyz="${forearm_length} 0 0"
-			rpy="0 0 0 " />
-		<parent link="left_forearm" />
-		<child link="left_grip" />
-		<axis xyz="0 0 1" />
-		<limit
-			lower="${-joint_limit}"
-			upper="${joint_limit}"
-			effort="${joint_effort}"
-			velocity="${joint_velocity}" />
-		<dynamics
-			damping="0"
-			friction="0" />
-	</joint>
 	<link name="left_grip">
 		<inertial>
@@ -391,9 +166,9 @@
 			<mass value="${gripper_mass}" />
 			<inertia
-				ixx="0.000001"
-				ixy="0.000001"
-				ixz="0.000001"
-				iyy="0.000001"
-				iyz="0.000001"
+				ixx="0.0001"
+				ixy="0.0001"
+				ixz="0.0001"
+				iyy="0.0001"
+				iyz="0.0001"
 				izz="${gripper_inertia}" />
 		</inertial>
@@ -414,46 +189,18 @@
 				<box size="${gripper_length} 0.02 0.02"/>
 			</geometry>
-			<surface>
+			<!-- <surface>
 				<friction>
 					<ode>
-						<mu>0</mu>           <!-- Coefficient of friction -->
-						<mu2>0</mu2>         <!-- Secondary coefficient of friction -->
+						<mu>0</mu>
+						<mu2>0</mu2>
 					</ode>
 				</friction>
-			</surface>
+			</surface> -->
 		</collision>
-		<!-- <xacro:inertial_box mass="0.046" x="0.0672" y="0.02" z="0.02">
-			<origin xyz="${gripper_length/2} 0 0" rpy="0 0 0"/>
-		</xacro:inertial_box> -->
-		<!-- <gazebo>
-			<sensor type="imu" name="imu_sensor">
-				<always_on>true</always_on>
-				<update_rate>100.0</update_rate>
-				<imu>
-					<angular_velocity>
-					<x>true</x>
-					<y>true</y>
-					<z>true</z>
-					</angular_velocity>
-					<linear_acceleration>
-					<x>true</x>
-					<y>true</y>
-					<z>true</z>
-					</linear_acceleration>
-				</imu>
-				<plugin name="imu_plugin" filename="libgazebo_ros_imu.so">
-					<ros>
-					<namespace>/cepheus</namespace>
-					<remapping>imu/data:=/imu/data</remapping>
-					</ros>
-					<robotNamespace>/cepheus</robotNamespace>
-					<topicName>imu</topicName>
-					<frameName>left_grip</frameName>
-					<updateRate>100</updateRate>
-					<initialOrientationAsReference>false</initialOrientationAsReference>
-				</plugin>
-			</sensor>
-		</gazebo> -->
-	</link>
+	</link>
+    <gazebo reference="left_grip">
+		<mu1>0</mu1>
+		<mu2>0</mu2>
+	</gazebo>
 	<joint name="final_joint" type="revolute">
 		<parent link="left_grip"/>
@@ -462,5 +209,5 @@
 			xyz="${gripper_length} 0 0"
 			rpy="0 0 0 " />
-		<axis xyz="1 0 0"/>
+		<axis xyz="0 1 0"/>
 		<limit lower="-1" upper="1" effort="${joint_effort}" velocity="${joint_velocity}"/>
 		<dynamics damping="1" friction="1"/>
@@ -509,16 +256,5 @@
 		</plugin>
 	</gazebo>
-	<gazebo>
-		<plugin filename="libgazebo_ros_force.so" name="gazebo_ros_force" >
-			<!-- <alwaysOn>true</alwaysOn> -->
-			<!-- <update>100</update> -->
-			<!-- <updateRate>0</updateRate> anti gia 100 -->
-			<bodyName>cepheus_base</bodyName>
-			<topicName>force_base_topic</topicName>
-			<force_reference_frame>cepheus_base</force_reference_frame>
-		</plugin>
-	</gazebo>
 	<gazebo reference="left_grip">
-		<gravity>false</gravity>
 		<sensor name="imu_sensor" type="imu">
 			<always_on>true</always_on>
@@ -539,4 +275,3 @@
 		</sensor>
   </gazebo>
-	<!-- <gravity>false</gravity> -->
 </robot>
