Commit message: eftiaksa diko mou peirama

File: src/cepheus_description/urdf/cepheus_simplified.xacro (robot description, xacro)
@@ -3,8 +3,22 @@
 	<xacro:include filename="$(find cepheus_description)/urdf/cepheus.gazebo" />
 	<xacro:include filename="$(find cepheus_description)/urdf/materials.xacro" />
+	<xacro:include filename="$(find cepheus_description)/urdf/inertial_macros.xacro"/>
 	<xacro:property name="camera_link" value="0.05" /> <!-- Size of square 'camera' box -->
-	<xacro:property name="arm" value="0.37" />
+	<!-- <xacro:property name="arm" value="0.37" />
 	<xacro:property name="forearm" value="0.286" />
-	<xacro:property name="gripper" value="0.0672" />
+	<xacro:property name="gripper" value="0.0672" /> -->
+	<xacro:property name="base_radius" value="0.2" />
+	<xacro:property name="y" value="0.02" />
+	<xacro:property name="arm_length" value="0.5" />
+	<xacro:property name="forearm_length" value="0.5" />
+	<xacro:property name="gripper_length" value="0.25" />
+	<xacro:property name="base_mass" value="53" />
+	<xacro:property name="arm_mass" value="1" />
+	<xacro:property name="forearm_mass" value="0.5" />
+	<xacro:property name="gripper_mass" value="0.1" />
+	<xacro:property name="base_inertia" value="${(1/2)*base_mass*base_radius*base_radius}" />
+	<xacro:property name="arm_inertia" value="${(1/12)*arm_mass*(arm_length*arm_length+y*y)}" />
+	<xacro:property name="forearm_inertia" value="${(1/12)*forearm_mass*(forearm_length*forearm_length+y*y)}" />
+	<xacro:property name="gripper_inertia" value="${(1/12)*gripper_mass*(gripper_length*gripper_length+y*y)}" />
 	<link name="world">
 		<!-- <joint name="world_joint" type="continuous">
@@ -39,8 +53,8 @@
 			<inertia
 				ixx="1e-2"
-				ixy="0.0"
-				ixz="0.0"
+				ixy="0.0001"
+				ixz="0.0001"
 				iyy="1e-2"
-				iyz="0.0"
+				iyz="0.0001"
 				izz="1e-2" />
 		</inertial>
@@ -81,8 +95,8 @@
 			<inertia
 				ixx="1e-2"
-				ixy="0.0"
-				ixz="0.0"
+				ixy="0.0001"
+				ixz="0.0001"
 				iyy="1e-2"
-				iyz="0.0"
+				iyz="0.0001"
 				izz="1e-2" />
 		</inertial>
@@ -118,25 +132,38 @@
 		<child link="cepheus_base"/>
 	</joint>
+	<transmission name="tran1">
+		<type>
+			transmission_interface/SimpleTransmission</type>
+		<joint name="r_joint">
+			<hardwareInterface>hardware_interface/EffortJointInterface</hardwareInterface>
+		</joint>
+		<actuator name="motor1">
+			<hardwareInterface>EffortJointInterface</hardwareInterface>
+			<mechanicalReduction>1</mechanicalReduction>
+		</actuator>
+	</transmission>
 	<!-- extra links addition END -->
 	<link name="cepheus_base">
-		<inertial>
-			<origin
-				xyz="0.0024 0.02937 0.15711"
-				rpy="0 0 0" />
-			<mass value="53" />
-			<inertia
-				ixx="0"
-				ixy="0"
-				ixz="0"
-				iyy="0"
-				iyz="0"
-				izz="2.1837" />
+		<!-- <xacro:inertial_cylinder mass="53" length="0.43" radius="0.2">
+			<origin xyz="0.0024 0.02937 0.15711" rpy="0 0 0 "/>
+		</xacro:inertial_cylinder> -->
+		<inertial>
+			<origin xyz="0.0024 0.02937 0.15711" rpy="0 0 0" />
+			<mass value="${base_mass}"/>
+			<inertia
+				ixx="0.000001"
+				ixy="0.000001"
+				ixz="0.000001"
+				iyy="0.000001"
+				iyz="0.000001"
+				izz="${base_inertia}" />
 		</inertial>
 		<visual>
 			<origin
-				xyz="0 0 0"
-				rpy="0 0 0" />
-			<geometry>
-				<mesh filename="package://cepheus_description/urdf/meshes/cepheus.STL" />
+				xyz="0 0 0.215"
+				rpy="0 0 0" />
+			<geometry>
+				<!-- <mesh filename="package://cepheus_description/urdf/meshes/cepheus.STL" /> -->
+				<cylinder length="0.43" radius="${base_radius}"/>
 			</geometry>
 			<material name="LightGrey"/>
@@ -147,9 +174,9 @@
 				rpy="0 0 0" />
 			<geometry>
-				<cylinder length="0.43" radius="0.2"/>
+				<cylinder length="0.43" radius="${base_radius}"/>
 			</geometry>
 		</collision>
 	</link>
-	<joint name="reaction_wheel_joint" type="continuous">
+	<!-- <joint name="reaction_wheel_joint" type="continuous">
 		<parent link="cepheus_base"/>
 		<child link="reaction_wheel"/>
@@ -169,19 +196,19 @@
 		<inertial>
 			<origin xyz="0 0 0.025" rpy="0 0 0" />
-			<mass value="1"/>
-			<inertia
-				ixx="0"
-				ixy="0"
-				ixz="0"
-				iyy="0"
-				iyz="0"
-				izz="0.00197" />
-		</inertial>
-	</link>
+			<mass value="0.1"/>
+			<inertia
+				ixx="0.0001"
+				ixy="0.0001"
+				ixz="0.0001"
+				iyy="0.0001"
+				iyz="0.0001"
+				izz="0.000197" />
+		</inertial>
+	</link> -->
 	<gazebo reference="cepheus_base">
 		<mu1>0</mu1>
 		<mu2>0</mu2>
 	</gazebo>
-	<transmission name="tran1">
+	<!-- <transmission name="tran1">
 		<type>
 			transmission_interface/SimpleTransmission</type>
@@ -193,5 +220,5 @@
 			<mechanicalReduction>1</mechanicalReduction>
 		</actuator>
-	</transmission>
+	</transmission> -->
 	<joint name="left_shoulder_joint" type="revolute">
 		<origin
@@ -202,6 +229,6 @@
 		<axis xyz="0 0 1" />
 		<limit
-			lower="-0.86"
-			upper="2.54"
+			lower="-1.57"
+			upper="1.57"
 			effort="20"
 			velocity="20" />
@@ -213,21 +240,21 @@
 		<inertial>
 			<origin
-				xyz="${arm/2} 0 0"
-				rpy="0 0 0" />
-			<mass value="0.2314" />
-			<inertia
-				ixx="0"
-				ixy="0"
-				ixz="0"
-				iyy="0"
-				iyz="0"
-				izz="0.00681" />
+				xyz="${arm_length/2} 0 0"
+				rpy="0 0 0" />
+			<mass value="${arm_mass}" />
+			<inertia
+				ixx="0.0001"
+				ixy="0.0001"
+				ixz="0.0001"
+				iyy="0.0001"
+				iyz="0.0001"
+				izz="${arm_inertia}" />
 		</inertial>
 		<visual>
 			<origin
-				xyz="${arm/2} 0 0"
-				rpy="0 0 0" />
-			<geometry>
-				<box size="${arm} 0.02 0.02" />
+				xyz="${arm_length/2} 0 0"
+				rpy="0 0 0" />
+			<geometry>
+				<box size="${arm_length} 0.02 0.02" />
 			</geometry>
 			<material name="LightGrey"/>
@@ -235,10 +262,13 @@
 		<collision>
 			<origin
-				xyz="${arm/2} 0.0 0"
-				rpy="0 0 0" />
-			<geometry>
-				<box size="${arm} 0.02 0.02"/>
+				xyz="${arm_length/2} 0.0 0"
+				rpy="0 0 0" />
+			<geometry>
+				<box size="${arm_length} 0.02 0.02"/>
 			</geometry>
 		</collision>
+		<!-- <xacro:inertial_box mass="0.2314" x="0.37" y="0.02" z="0.02">
+			<origin xyz="0.185 0 0" rpy="0 0 0"/>
+		</xacro:inertial_box> -->
 	</link>
 	<transmission name="tran2">
@@ -254,5 +284,5 @@
 	<joint name="left_elbow_joint" type="revolute">
 		<origin
-			xyz="${arm} 0 0"
+			xyz="${arm_length} 0 0"
 			rpy="0 0 0" />
 		<parent link="left_arm" />
@@ -271,21 +301,21 @@
 		<inertial>
 			<origin
-				xyz="${forearm/2} 0 0"
-				rpy="0 0 0" />
-			<mass value="0.1" />
-			<inertia
-				ixx="0"
-				ixy="0"
-				ixz="0"
-				iyy="0"
-				iyz="0"
-				izz="0.00001487" />
+				xyz="${forearm_length/2} 0 0"
+				rpy="0 0 0" />
+			<mass value="${forearm_mass}" />
+			<inertia
+				ixx="0.00001"
+				ixy="0.00001"
+				ixz="0.00001"
+				iyy="0.00001"
+				iyz="0.00001"
+				izz="${forearm_inertia}" />
 		</inertial>
 		<visual>
 			<origin
-				xyz="${forearm/2} 0 0"
-				rpy="0 0 0" />
-			<geometry>
-				<box size="${forearm} 0.02 0.02"/>
+				xyz="${forearm_length/2} 0 0"
+				rpy="0 0 0" />
+			<geometry>
+				<box size="${forearm_length} 0.02 0.02"/>
 			</geometry>
 			<material name="LightGrey"/>
@@ -293,10 +323,13 @@
 		<collision>
 			<origin
-				xyz="${forearm/2} 0 0"
-				rpy="0 0 0" />
-			<geometry>
-				<box size="${forearm} 0.02 0.02"/>
+				xyz="${forearm_length/2} 0 0"
+				rpy="0 0 0" />
+			<geometry>
+				<box size="${forearm_length} 0.02 0.02"/>
 			</geometry>
 		</collision>
+		<!-- <xacro:inertial_box mass="0.1" x="0.286" y="0.02" z="0.02">
+			<origin xyz="0.143 0 0" rpy="0 0 0"/>
+		</xacro:inertial_box> -->
 	</link>
 	<transmission name="tran3">
@@ -312,5 +345,5 @@
 	<joint name="left_wrist_joint" type="revolute">
 		<origin
-			xyz="${forearm} 0 0"
+			xyz="${forearm_length} 0 0"
 			rpy="0 0 0 " />
 		<parent link="left_forearm" />
@@ -320,6 +353,6 @@
 			lower="-1.570796327"
 			upper="1.570796327"
-			effort="1"
-			velocity="10" />
+			effort="2"
+			velocity="20" />
 		<dynamics
 			damping="1"
@@ -329,21 +362,21 @@
 		<inertial>
 			<origin
-				xyz="${gripper/2} 0 0"
-				rpy="0 0 0" />
-			<mass value="0.046" />
-			<inertia
-				ixx="0.0926325136613974"
-				ixy="-0.00333421740190982"
-				ixz="0.00529966557344093"
-				iyy="0.0752633235560557"
-				iyz="0.00191940596202769"
-				izz="0.000012287" />
+				xyz="${gripper_length/2} 0 0"
+				rpy="0 0 0" />
+			<mass value="${gripper_mass}" />
+			<inertia
+				ixx="0.000001"
+				ixy="0.000001"
+				ixz="0.000001"
+				iyy="0.000001"
+				iyz="0.000001"
+				izz="${gripper_inertia}" />
 		</inertial>
 		<visual>
 			<origin
-				xyz="${gripper/2} 0 0"
-				rpy="0 0 0" />
-			<geometry>
-				<box size="${gripper} 0.02 0.02"/>
+				xyz="${gripper_length/2} 0 0"
+				rpy="0 0 0" />
+			<geometry>
+				<box size="${gripper_length} 0.02 0.02"/>
 			</geometry>
 			<material name="LightGrey"/>
@@ -351,10 +384,13 @@
 		<collision>
 			<origin
-				xyz="${gripper/2} 0 0"
-				rpy="0 0 0" />
-			<geometry>
-				<box size="${gripper} 0.02 0.02"/>
+				xyz="${gripper_length/2} 0 0"
+				rpy="0 0 0" />
+			<geometry>
+				<box size="${gripper_length} 0.02 0.02"/>
 			</geometry>
 		</collision>
+		<!-- <xacro:inertial_box mass="0.046" x="0.0672" y="0.02" z="0.02">
+			<origin xyz="${gripper_length/2} 0 0" rpy="0 0 0"/>
+		</xacro:inertial_box> -->
 	</link>
 	<transmission name="tran4">
@@ -393,5 +429,5 @@
 			<bodyName>cepheus_base</bodyName>
 			<topicName>force_base_topic</topicName>
-			<force_reference_frame>world</force_reference_frame>
+			<force_reference_frame>cepheus_base</force_reference_frame>
 		</plugin>
 	</gazebo>

File: src/cepheus_description/urdf/simple_ring.xacro (robot description, xacro)
@@ -117,5 +117,5 @@
     <inertial>
       <mass value="1.0"/>
-      <inertia ixx="0.00833" ixy="0" ixz="0" iyy="0.00833" iyz="0" izz="0.00833"/>
+      <inertia ixx="0.00135" ixy="0" ixz="0" iyy="0.00135" iyz="0" izz="0.00135"/>
     </inertial>
   </link>

Commit message: afhsa th vash alla rw anenergh

File: src/cepheus_description/urdf/cepheus_simplified.xacro (robot description, xacro)
@@ -161,9 +161,9 @@
 		<visual>
 			<origin
-				xyz="0 0 0.215"
-				rpy="0 0 0" />
-			<geometry>
-				<!-- <mesh filename="package://cepheus_description/urdf/meshes/cepheus.STL" /> -->
-				<cylinder length="0.43" radius="${base_radius}"/>
+				xyz="0 0 0"
+				rpy="0 0 0" />
+			<geometry>
+				<mesh filename="package://cepheus_description/urdf/meshes/cepheus.STL" />
+				<!-- <cylinder length="0.43" radius="${base_radius}"/> -->
 			</geometry>
 			<material name="LightGrey"/>
@@ -178,5 +178,5 @@
 		</collision>
 	</link>
-	<!-- <joint name="reaction_wheel_joint" type="continuous">
+	<joint name="reaction_wheel_joint" type="continuous">
 		<parent link="cepheus_base"/>
 		<child link="reaction_wheel"/>
@@ -205,5 +205,5 @@
 				izz="0.000197" />
 		</inertial>
-	</link> -->
+	</link>
 	<gazebo reference="cepheus_base">
 		<mu1>0</mu1>

Commit message: xalasan ta x,y

File: src/cepheus_description/urdf/cepheus_simplified.xacro (robot description, xacro)
@@ -10,7 +10,7 @@
 	<xacro:property name="base_radius" value="0.2" />
 	<xacro:property name="y" value="0.02" />
-	<xacro:property name="arm_length" value="0.5" />
+	<!-- <xacro:property name="arm_length" value="0.5" />
 	<xacro:property name="forearm_length" value="0.5" />
-	<xacro:property name="gripper_length" value="0.25" />
+	<xacro:property name="gripper_length" value="0.125" />
 	<xacro:property name="base_mass" value="53" />
 	<xacro:property name="arm_mass" value="1" />
@@ -20,5 +20,17 @@
 	<xacro:property name="arm_inertia" value="${(1/12)*arm_mass*(arm_length*arm_length+y*y)}" />
 	<xacro:property name="forearm_inertia" value="${(1/12)*forearm_mass*(forearm_length*forearm_length+y*y)}" />
-	<xacro:property name="gripper_inertia" value="${(1/12)*gripper_mass*(gripper_length*gripper_length+y*y)}" />
+	<xacro:property name="gripper_inertia" value="${(1/12)*gripper_mass*(gripper_length*gripper_length+y*y)}" /> -->
+	<!-- gia sygkrish me simscape 29/7 -->
+	<xacro:property name="arm_length" value="0.37" />
+	<xacro:property name="forearm_length" value="0.368" />
+	<xacro:property name="gripper_length" value="0.0822" />
+	<xacro:property name="base_mass" value="53" />
+	<xacro:property name="arm_mass" value="0.2314" />
+	<xacro:property name="forearm_mass" value="0.1" />
+	<xacro:property name="gripper_mass" value="0.046" />
+	<xacro:property name="base_inertia" value="2.1837" />
+	<xacro:property name="arm_inertia" value="0.0068" />
+	<xacro:property name="forearm_inertia" value="${1.487/100000}" />
+	<xacro:property name="gripper_inertia" value="${1.2287/100000}" />
 	<link name="world">
 		<!-- <joint name="world_joint" type="continuous">
@@ -161,9 +173,9 @@
 		<visual>
 			<origin
-				xyz="0 0 0"
-				rpy="0 0 0" />
-			<geometry>
-				<mesh filename="package://cepheus_description/urdf/meshes/cepheus.STL" />
-				<!-- <cylinder length="0.43" radius="${base_radius}"/> -->
+				xyz="0 0 0.215"
+				rpy="0 0 0" />
+			<geometry>
+				<!-- <mesh filename="package://cepheus_description/urdf/meshes/cepheus.STL" /> -->
+				<cylinder length="0.43" radius="${base_radius}"/>
 			</geometry>
 			<material name="LightGrey"/>
@@ -178,5 +190,5 @@
 		</collision>
 	</link>
-	<joint name="reaction_wheel_joint" type="continuous">
+	<!-- <joint name="reaction_wheel_joint" type="continuous">
 		<parent link="cepheus_base"/>
 		<child link="reaction_wheel"/>
@@ -205,5 +217,5 @@
 				izz="0.000197" />
 		</inertial>
-	</link>
+	</link> -->
 	<gazebo reference="cepheus_base">
 		<mu1>0</mu1>
@@ -404,4 +416,10 @@
 		</actuator>
 	</transmission>
+	<gazebo reference="left_wrist_joint">
+		<provideFeedback>true</provideFeedback>
+		<!-- <sensor name="force_torque" type="force_torque">
+          <update_rate>30</update_rate>
+    	</sensor> -->
+	</gazebo>
     <gazebo>
 		<plugin name="ft_sensor" filename="libgazebo_ros_ft_sensor.so">
@@ -416,10 +434,4 @@
 		</plugin>
 	</gazebo>
-    <gazebo reference="left_wrist_joint">
-		<provideFeedback>true</provideFeedback>
-		<!-- <sensor name="force_torque" type="force_torque">
-          <update_rate>30</update_rate>
-    	</sensor> -->
-	</gazebo>
 	<gazebo>
 		<plugin filename="libgazebo_ros_force.so" name="gazebo_ros_force" >

Commit message: eftiaksa to urdf gia damping friction, base PD doulevei

File: src/cepheus_description/urdf/cepheus_simplified.xacro (robot description, xacro)
@@ -33,4 +33,6 @@
 	<xacro:property name="forearm_inertia" value="${1.487/100000}" />
 	<xacro:property name="gripper_inertia" value="${1.2287/100000}" />
+	<xacro:property name="joint_damping" value="0.1" />
+	<xacro:property name="joint_friction" value="0.1" />
 	<link name="world">
 		<!-- <joint name="world_joint" type="continuous">
@@ -55,5 +57,5 @@
 		<axis xyz="1 0 0"/>
 		<limit lower="-100" upper="100" effort="1000" velocity="10000"/>
-		<dynamics damping="0" friction="0"/>
+		<dynamics damping="${joint_damping}" friction="${joint_friction}"/>
 	</joint>
 	<link name="p1">
@@ -96,6 +98,6 @@
 			velocity="10000"/>
 		<dynamics
-			damping="0"
-			friction="0"/>
+			damping="${joint_damping}"
+			friction="${joint_friction}"/>
 	</joint>
 	<link name="p2">
@@ -246,6 +248,6 @@
 			velocity="20" />
 		<dynamics
-			damping="1"
-			friction="1" />
+			damping="${joint_damping}"
+			friction="${joint_friction}" />
 	</joint>
 	<link name="left_arm">
@@ -307,6 +309,6 @@
 			velocity="20" />
 		<dynamics
-			damping="1"
-			friction="1" />
+			damping="${joint_damping}"
+			friction="${joint_friction}" />
 	</joint>
 	<link name="left_forearm">
@@ -368,6 +370,6 @@
 			velocity="20" />
 		<dynamics
-			damping="1"
-			friction="1" />
+			damping="${joint_damping}"
+			friction="${joint_friction}" />
 	</joint>
 	<link name="left_grip">

Commit message: spaei to gazebo

File: src/cepheus_description/urdf/cepheus_simplified.xacro (robot description, xacro)
@@ -192,5 +192,5 @@
 		</collision>
 	</link>
-	<!-- <joint name="reaction_wheel_joint" type="continuous">
+	<joint name="reaction_wheel_joint" type="continuous">
 		<parent link="cepheus_base"/>
 		<child link="reaction_wheel"/>
@@ -210,5 +210,5 @@
 		<inertial>
 			<origin xyz="0 0 0.025" rpy="0 0 0" />
-			<mass value="0.1"/>
+			<mass value="1"/>
 			<inertia
 				ixx="0.0001"
@@ -219,10 +219,10 @@
 				izz="0.000197" />
 		</inertial>
-	</link> -->
+	</link>
 	<gazebo reference="cepheus_base">
 		<mu1>0</mu1>
 		<mu2>0</mu2>
 	</gazebo>
-	<!-- <transmission name="tran1">
+	<transmission name="tran1">
 		<type>
 			transmission_interface/SimpleTransmission</type>
@@ -234,5 +234,5 @@
 			<mechanicalReduction>1</mechanicalReduction>
 		</actuator>
-	</transmission> -->
+	</transmission>
 	<joint name="left_shoulder_joint" type="revolute">
 		<origin

Commit message: kanei svoures

File: src/cepheus_description/urdf/cepheus_simplified.xacro (robot description, xacro)
@@ -195,5 +195,6 @@
 		<parent link="cepheus_base"/>
 		<child link="reaction_wheel"/>
-		<origin xyz="0.065 0 0.03815" rpy="0 0 0"/>
+		<!-- <origin xyz="0.065 0 0.03815" rpy="0 0 0"/> -->
+		<origin xyz="0 0 0.03815" rpy="0 0 0 "/>
 		<axis xyz="0 0 1" />
 	</joint>

Commit message: doulevei to free space se mikra tf

File: src/cepheus_description/urdf/cepheus_simplified.xacro (robot description, xacro)
@@ -33,6 +33,6 @@
 	<xacro:property name="forearm_inertia" value="${1.487/100000}" />
 	<xacro:property name="gripper_inertia" value="${1.2287/100000}" />
-	<xacro:property name="joint_damping" value="0.1" />
-	<xacro:property name="joint_friction" value="0.1" />
+	<xacro:property name="joint_damping" value="0.01" />
+	<xacro:property name="joint_friction" value="0.01" />
 	<link name="world">
 		<!-- <joint name="world_joint" type="continuous">

Commit message: isos ftaine oi arxikes synthikes

File: src/cepheus_description/urdf/cepheus_simplified.xacro (robot description, xacro)
@@ -33,6 +33,6 @@
 	<xacro:property name="forearm_inertia" value="${1.487/100000}" />
 	<xacro:property name="gripper_inertia" value="${1.2287/100000}" />
-	<xacro:property name="joint_damping" value="0.01" />
-	<xacro:property name="joint_friction" value="0.01" />
+	<xacro:property name="joint_damping" value="0.001" />
+	<xacro:property name="joint_friction" value="0.001" />
 	<link name="world">
 		<!-- <joint name="world_joint" type="continuous">

File: src/cepheus_description/urdf/simple_ring.xacro (robot description, xacro)
@@ -105,5 +105,5 @@
         <box size="0.09 0.09 0.09"/>
       </geometry>
-      <!-- <origin xyz="5 0 0" /> -->
+      <origin xyz="0.045 0 0" rpy="0 0 0" />
       <material name="blue">
         <color rgba="0 0 .8 1"/>

Commit message: free space done

File: src/cepheus_description/urdf/cepheus_simplified.xacro (robot description, xacro)
@@ -81,5 +81,5 @@
 		<type>transmission_interface/SimpleTransmission</type>
 		<joint name="p1_joint">
-			<hardwareInterface>hardware_interface/EffortJointInterface</hardwareInterface>
+			<hardwareInterface>EffortJointInterface</hardwareInterface>
 		</joint>
 		<actuator name="lin_motor1">
@@ -133,5 +133,5 @@
 		<type>transmission_interface/SimpleTransmission</type>
 		<joint name="p2_joint">
-			<hardwareInterface>hardware_interface/EffortJointInterface</hardwareInterface>
+			<hardwareInterface>EffortJointInterface</hardwareInterface>
 		</joint>
 		<actuator name="lin_motor2">
@@ -145,4 +145,5 @@
 		<origin rpy="0 0 0" xyz="0 0 0"/>
 		<child link="cepheus_base"/>
+		<dynamics damping="${joint_damping}" friction="${joint_friction}"/>
 	</joint>
 	<transmission name="tran1">
@@ -150,5 +151,5 @@
 			transmission_interface/SimpleTransmission</type>
 		<joint name="r_joint">
-			<hardwareInterface>hardware_interface/EffortJointInterface</hardwareInterface>
+			<hardwareInterface>EffortJointInterface</hardwareInterface>
 		</joint>
 		<actuator name="motor1">
@@ -198,4 +199,5 @@
 		<origin xyz="0 0 0.03815" rpy="0 0 0 "/>
 		<axis xyz="0 0 1" />
+		<dynamics damping="${joint_damping}" friction="${joint_friction}"/>
 	</joint>
 	<link name="reaction_wheel">
@@ -229,5 +231,5 @@
 			transmission_interface/SimpleTransmission</type>
 		<joint name="reaction_wheel_joint">
-			<hardwareInterface>hardware_interface/EffortJointInterface</hardwareInterface>
+			<hardwareInterface>EffortJointInterface</hardwareInterface>
 		</joint>
 		<actuator name="motor1">
@@ -290,5 +292,5 @@
 		<type>transmission_interface/SimpleTransmission</type>
 		<joint name="left_shoulder_joint">
-			<hardwareInterface>hardware_interface/EffortJointInterface</hardwareInterface>
+			<hardwareInterface>EffortJointInterface</hardwareInterface>
 		</joint>
 		<actuator name="motor2">
@@ -351,5 +353,5 @@
 		<type>transmission_interface/SimpleTransmission</type>
 		<joint name="left_elbow_joint">
-			<hardwareInterface>hardware_interface/EffortJointInterface</hardwareInterface>
+			<hardwareInterface>EffortJointInterface</hardwareInterface>
 		</joint>
 		<actuator name="motor3">
@@ -412,5 +414,5 @@
 		<type>transmission_interface/SimpleTransmission</type>
 		<joint name="left_wrist_joint">
-			<hardwareInterface>hardware_interface/EffortJointInterface</hardwareInterface>
+			<hardwareInterface>EffortJointInterface</hardwareInterface>
 		</joint>
 		<actuator name="motor4">

File: src/cepheus_description/urdf/simple_ring.xacro (robot description, xacro)
@@ -114,8 +114,10 @@
         <box size="0.09 0.09 0.09"/>
       </geometry>
+	  <origin xyz="0.045 0 0" rpy="0 0 0" />
     </collision>
     <inertial>
       <mass value="1.0"/>
       <inertia ixx="0.00135" ixy="0" ixz="0" iyy="0.00135" iyz="0" izz="0.00135"/>
+	  <origin xyz="0.045 0 0" rpy="0 0 0" />
     </inertial>
   </link>
