Commit message: thelei sostes arx sinth

File: src/cepheus_description/urdf/cepheus_simplified.xacro (robot description, xacro)
@@ -81,8 +81,8 @@
 		<type>transmission_interface/SimpleTransmission</type>
 		<joint name="p1_joint">
-			<hardwareInterface>EffortJointInterface</hardwareInterface>
+			<hardwareInterface>hardware_interface/EffortJointInterface</hardwareInterface>
 		</joint>
 		<actuator name="lin_motor1">
-			<hardwareInterface>EffortJointInterface</hardwareInterface>
+			<hardwareInterface>hardware_interface/EffortJointInterface</hardwareInterface>
 			<mechanicalReduction>1</mechanicalReduction>
 		</actuator>
@@ -133,8 +133,8 @@
 		<type>transmission_interface/SimpleTransmission</type>
 		<joint name="p2_joint">
-			<hardwareInterface>EffortJointInterface</hardwareInterface>
+			<hardwareInterface>hardware_interface/EffortJointInterface</hardwareInterface>
 		</joint>
 		<actuator name="lin_motor2">
-			<hardwareInterface>EffortJointInterface</hardwareInterface>
+			<hardwareInterface>hardware_interface/EffortJointInterface</hardwareInterface>
 			<mechanicalReduction>1</mechanicalReduction>
 		</actuator>
@@ -151,8 +151,8 @@
 			transmission_interface/SimpleTransmission</type>
 		<joint name="r_joint">
-			<hardwareInterface>EffortJointInterface</hardwareInterface>
+			<hardwareInterface>hardware_interface/EffortJointInterface</hardwareInterface>
 		</joint>
 		<actuator name="motor1">
-			<hardwareInterface>EffortJointInterface</hardwareInterface>
+			<hardwareInterface>hardware_interface/EffortJointInterface</hardwareInterface>
 			<mechanicalReduction>1</mechanicalReduction>
 		</actuator>
@@ -231,8 +231,8 @@
 			transmission_interface/SimpleTransmission</type>
 		<joint name="reaction_wheel_joint">
-			<hardwareInterface>EffortJointInterface</hardwareInterface>
+			<hardwareInterface>hardware_interface/EffortJointInterface</hardwareInterface>
 		</joint>
 		<actuator name="motor1">
-			<hardwareInterface>EffortJointInterface</hardwareInterface>
+			<hardwareInterface>hardware_interface/EffortJointInterface</hardwareInterface>
 			<mechanicalReduction>1</mechanicalReduction>
 		</actuator>
@@ -292,8 +292,8 @@
 		<type>transmission_interface/SimpleTransmission</type>
 		<joint name="left_shoulder_joint">
-			<hardwareInterface>EffortJointInterface</hardwareInterface>
+			<hardwareInterface>hardware_interface/EffortJointInterface</hardwareInterface>
 		</joint>
 		<actuator name="motor2">
-			<hardwareInterface>EffortJointInterface</hardwareInterface>
+			<hardwareInterface>hardware_interface/EffortJointInterface</hardwareInterface>
 			<mechanicalReduction>1</mechanicalReduction>
 		</actuator>
@@ -353,8 +353,8 @@
 		<type>transmission_interface/SimpleTransmission</type>
 		<joint name="left_elbow_joint">
-			<hardwareInterface>EffortJointInterface</hardwareInterface>
+			<hardwareInterface>hardware_interface/EffortJointInterface</hardwareInterface>
 		</joint>
 		<actuator name="motor3">
-			<hardwareInterface>EffortJointInterface</hardwareInterface>
+			<hardwareInterface>hardware_interface/EffortJointInterface</hardwareInterface>
 			<mechanicalReduction>1</mechanicalReduction>
 		</actuator>
@@ -414,8 +414,8 @@
 		<type>transmission_interface/SimpleTransmission</type>
 		<joint name="left_wrist_joint">
-			<hardwareInterface>EffortJointInterface</hardwareInterface>
+			<hardwareInterface>hardware_interface/EffortJointInterface</hardwareInterface>
 		</joint>
 		<actuator name="motor4">
-			<hardwareInterface>EffortJointInterface</hardwareInterface>
+			<hardwareInterface>hardware_interface/EffortJointInterface</hardwareInterface>
 			<mechanicalReduction>1</mechanicalReduction>
 		</actuator>

File: src/cepheus_description/urdf/simple_ring.xacro (robot description, xacro)
@@ -117,6 +117,6 @@
     </collision>
     <inertial>
-      <mass value="1.0"/>
-      <inertia ixx="0.00135" ixy="0" ixz="0" iyy="0.00135" iyz="0" izz="0.00135"/>
+      <mass value="10.0"/>
+      <inertia ixx="0.0135" ixy="0" ixz="0" iyy="0.0135" iyz="0" izz="0.0135"/>
 	  <origin xyz="0.045 0 0" rpy="0 0 0" />
     </inertial>

Commit message: isos thelei filtro

File: src/cepheus_description/urdf/cepheus_simplified.xacro (robot description, xacro)
@@ -24,5 +24,5 @@
 	<xacro:property name="arm_length" value="0.37" />
 	<xacro:property name="forearm_length" value="0.368" />
-	<xacro:property name="gripper_length" value="0.0822" />
+	<xacro:property name="gripper_length" value="0.0411" />
 	<xacro:property name="base_mass" value="53" />
 	<xacro:property name="arm_mass" value="0.2314" />
@@ -32,5 +32,5 @@
 	<xacro:property name="arm_inertia" value="0.0068" />
 	<xacro:property name="forearm_inertia" value="${1.487/100000}" />
-	<xacro:property name="gripper_inertia" value="${1.2287/100000}" />
+	<xacro:property name="gripper_inertia" value="${9.61/100000}" />
 	<xacro:property name="joint_damping" value="0.001" />
 	<xacro:property name="joint_friction" value="0.001" />
@@ -435,5 +435,5 @@
           		<type>gaussian</type>
           		<mean>0.0</mean>
-          		<stddev>0.003</stddev> <!-- change this to simulate noise -->
+          		<stddev>0.0003</stddev> <!-- change this to simulate noise -->
         	</noise>
 		</plugin>

File: src/cepheus_description/urdf/simple_ring.xacro (robot description, xacro)
@@ -117,6 +117,6 @@
     </collision>
     <inertial>
-      <mass value="10.0"/>
-      <inertia ixx="0.0135" ixy="0" ixz="0" iyy="0.0135" iyz="0" izz="0.0135"/>
+      <mass value="20.0"/>
+      <inertia ixx="0.027" ixy="0" ixz="0" iyy="0.027" iyz="0" izz="0.027"/>
 	  <origin xyz="0.045 0 0" rpy="0 0 0" />
     </inertial>

Commit message: kati xalasa

File: src/cepheus_description/urdf/cepheus_simplified.xacro (robot description, xacro)
@@ -33,6 +33,6 @@
 	<xacro:property name="forearm_inertia" value="${1.487/100000}" />
 	<xacro:property name="gripper_inertia" value="${9.61/100000}" />
-	<xacro:property name="joint_damping" value="0.001" />
-	<xacro:property name="joint_friction" value="0.001" />
+	<xacro:property name="joint_damping" value="0.01" />
+	<xacro:property name="joint_friction" value="0.01" />
 	<link name="world">
 		<!-- <joint name="world_joint" type="continuous">
@@ -246,6 +246,6 @@
 		<axis xyz="0 0 1" />
 		<limit
-			lower="-1.57"
-			upper="1.57"
+			lower="-3.14"
+			upper="3.14"
 			effort="20"
 			velocity="20" />
@@ -308,6 +308,6 @@
 		<limit
 			lower="-3.14"
-			upper="1.5"
-			effort="2"
+			upper="3.14"
+			effort="20"
 			velocity="20" />
 		<dynamics
@@ -368,7 +368,7 @@
 		<axis xyz="0 0 1" />
 		<limit
-			lower="-1.570796327"
-			upper="1.570796327"
-			effort="2"
+			lower="-3.14"
+			upper="3.14"
+			effort="20"
 			velocity="20" />
 		<dynamics

Commit message: eftiaksa ta plots na ftiakso ton xrono

File: src/cepheus_description/urdf/cepheus_simplified.xacro (robot description, xacro)
@@ -33,6 +33,7 @@
 	<xacro:property name="forearm_inertia" value="${1.487/100000}" />
 	<xacro:property name="gripper_inertia" value="${9.61/100000}" />
-	<xacro:property name="joint_damping" value="0.01" />
-	<xacro:property name="joint_friction" value="0.01" />
+	<xacro:property name="joint_damping" value="0.00001" />
+	<xacro:property name="joint_friction" value="0.00001" />
+	<xacro:property name="joint_limit" value="3.14" />
 	<link name="world">
 		<!-- <joint name="world_joint" type="continuous">
@@ -246,6 +247,6 @@
 		<axis xyz="0 0 1" />
 		<limit
-			lower="-3.14"
-			upper="3.14"
+			lower="${-joint_limit}"
+			upper="${joint_limit}"
 			effort="20"
 			velocity="20" />
@@ -307,6 +308,6 @@
 		<axis xyz="0 0 1" />
 		<limit
-			lower="-3.14"
-			upper="3.14"
+			lower="${-joint_limit}"
+			upper="${joint_limit}"
 			effort="20"
 			velocity="20" />
@@ -368,6 +369,6 @@
 		<axis xyz="0 0 1" />
 		<limit
-			lower="-3.14"
-			upper="3.14"
+			lower="${-joint_limit}"
+			upper="${joint_limit}"
 			effort="20"
 			velocity="20" />
@@ -410,4 +411,29 @@
 			<origin xyz="${gripper_length/2} 0 0" rpy="0 0 0"/>
 		</xacro:inertial_box> -->
+	</link>
+	<joint name="final_joint" type="revolute">
+		<parent link="left_grip"/>
+		<child link="final_link"/>
+		<origin
+			xyz="${gripper_length} 0 0"
+			rpy="0 0 0 " />
+		<axis xyz="0 1 0"/>
+		<limit lower="-1" upper="1" effort="10" velocity="10000"/>
+		<dynamics damping="1" friction="1"/>
+	</joint>
+	<link name="final_link">
+		<inertial>
+			<origin
+				xyz="0.0 0.0 0.0"
+				rpy="0.0 0.0 0.0" />
+			<mass value="0.0001" />
+			<inertia
+				ixx="1e-6"
+				ixy="0.00001"
+				ixz="0.00001"
+				iyy="1e-6"
+				iyz="0.00001"
+				izz="1e-6" />
+		</inertial>
 	</link>
 	<transmission name="tran4">

Commit message: to live plot thelei fix

File: src/cepheus_description/urdf/cepheus_simplified.xacro (robot description, xacro)
@@ -33,6 +33,6 @@
 	<xacro:property name="forearm_inertia" value="${1.487/100000}" />
 	<xacro:property name="gripper_inertia" value="${9.61/100000}" />
-	<xacro:property name="joint_damping" value="0.00001" />
-	<xacro:property name="joint_friction" value="0.00001" />
+	<xacro:property name="joint_damping" value="0.001" />
+	<xacro:property name="joint_friction" value="0.001" />
 	<xacro:property name="joint_limit" value="3.14" />
 	<link name="world">

Commit message: ti na po

File: src/cepheus_description/urdf/cepheus_simplified.xacro (robot description, xacro)
@@ -214,5 +214,5 @@
 		<inertial>
 			<origin xyz="0 0 0.025" rpy="0 0 0" />
-			<mass value="1"/>
+			<mass value="0.001"/>
 			<inertia
 				ixx="0.0001"

Commit message: fixed git

File: src/cepheus_description/urdf/cepheus_simplified.xacro (robot description, xacro)
@@ -24,5 +24,6 @@
 	<xacro:property name="arm_length" value="0.37" />
 	<xacro:property name="forearm_length" value="0.368" />
-	<xacro:property name="gripper_length" value="0.0411" />
+	<!-- <xacro:property name="gripper_length" value="0.0411" /> -->
+	<xacro:property name="gripper_length" value="0.0822" />
 	<xacro:property name="base_mass" value="53" />
 	<xacro:property name="arm_mass" value="0.2314" />
@@ -32,5 +33,6 @@
 	<xacro:property name="arm_inertia" value="0.0068" />
 	<xacro:property name="forearm_inertia" value="${1.487/100000}" />
-	<xacro:property name="gripper_inertia" value="${9.61/100000}" />
+	<!-- <xacro:property name="gripper_inertia" value="${9.61/100000}" /> -->
+	<xacro:property name="gripper_inertia" value="${1.2287/100000}" />
 	<xacro:property name="joint_damping" value="0.001" />
 	<xacro:property name="joint_friction" value="0.001" />
@@ -194,13 +196,12 @@
 		</collision>
 	</link>
-	<joint name="reaction_wheel_joint" type="continuous">
+	<!-- <joint name="reaction_wheel_joint" type="continuous">
 		<parent link="cepheus_base"/>
 		<child link="reaction_wheel"/>
-		<!-- <origin xyz="0.065 0 0.03815" rpy="0 0 0"/> -->
 		<origin xyz="0 0 0.03815" rpy="0 0 0 "/>
 		<axis xyz="0 0 1" />
 		<dynamics damping="${joint_damping}" friction="${joint_friction}"/>
-	</joint>
-	<link name="reaction_wheel">
+	</joint> -->
+	<!-- <link name="reaction_wheel">
 		<visual>
 			<material name="silver">
@@ -223,10 +224,10 @@
 				izz="0.000197" />
 		</inertial>
-	</link>
+	</link> -->
 	<gazebo reference="cepheus_base">
 		<mu1>0</mu1>
 		<mu2>0</mu2>
 	</gazebo>
-	<transmission name="tran1">
+	<!-- <transmission name="tran1">
 		<type>
 			transmission_interface/SimpleTransmission</type>
@@ -238,5 +239,5 @@
 			<mechanicalReduction>1</mechanicalReduction>
 		</actuator>
-	</transmission>
+	</transmission> -->
 	<joint name="left_shoulder_joint" type="revolute">
 		<origin
@@ -429,10 +430,10 @@
 			<mass value="0.0001" />
 			<inertia
-				ixx="1e-6"
+				ixx="1e-7"
 				ixy="0.00001"
 				ixz="0.00001"
-				iyy="1e-6"
+				iyy="1e-7"
 				iyz="0.00001"
-				izz="1e-6" />
+				izz="1e-7" />
 		</inertial>
 	</link>

Commit message: kalh prosomoiosh

File: src/cepheus_description/urdf/cepheus_simplified.xacro (robot description, xacro)
@@ -414,12 +414,18 @@
 				<box size="${gripper_length} 0.02 0.02"/>
 			</geometry>
-			<surface>
+			<!-- <surface>
 				<friction>
 					<ode>
-						<mu>0</mu>           <!-- Coefficient of friction -->
-						<mu2>0</mu2>         <!-- Secondary coefficient of friction -->
+						<mu>0</mu>
+						<mu2>0</mu2>
 					</ode>
 				</friction>
-			</surface>
+				<contact>
+        			<ode>
+						<kp>1000000.0</kp>
+						<kd>0.0</kd>
+					</ode>
+				</contact>
+			</surface> -->
 		</collision>
 		<!-- <xacro:inertial_box mass="0.046" x="0.0672" y="0.02" z="0.02">
@@ -460,5 +466,5 @@
 		<child link="final_link"/>
 		<origin
-			xyz="${gripper_length} 0 0"
+			xyz="${gripper_length} 0 0.02"
 			rpy="0 0 0 " />
 		<axis xyz="1 0 0"/>
@@ -538,4 +544,6 @@
 			<!-- <pose>0 0 0 0 0 0</pose> -->
 		</sensor>
+		<kp>1000000</kp>
+		<kd>0</kd>
   </gazebo>
 	<!-- <gravity>false</gravity> -->

File: src/cepheus_description/urdf/simple_ring.xacro (robot description, xacro)
@@ -1,9 +1,10 @@
 <?xml version="1.0"?>
 <robot xmlns:xacro="http://www.ros.org/wiki/xacro" name="simple_ring">
-  <xacro:include filename="$(find cepheus_description)/urdf/simple_ring.gazebo" />
-  <link name="world"></link>
-	<!-- <joint name="p1_joint" type="prismatic">
+	<xacro:include filename="$(find cepheus_description)/urdf/simple_ring.gazebo" />
+	<link name="world"></link>
+	<joint name="p1_joint" type="prismatic">
 		<parent link="world"/>
 		<child link="p1"/>
+		<origin rpy="0 0 0" xyz="0 0 0.045"/>
 		<axis xyz="1 0 0"/>
 		<limit lower="-100" upper="100" effort="1000" velocity="10000"/>
@@ -15,11 +16,11 @@
 				xyz="0.0 0.0 0.0"
 				rpy="0.0 0.0 0.0" />
-			<mass value="0.01" />
+			<mass value="0.001" />
 			<inertia
 				ixx="1e-2"
-				ixy="0.0"
-				ixz="0.0"
+				ixy="0.000001"
+				ixz="0.000001"
 				iyy="1e-2"
-				iyz="0.0"
+				iyz="0.000001"
 				izz="1e-2" />
 		</inertial>
@@ -29,14 +30,4 @@
 		<mu2>0</mu2>
 	</gazebo>
-	<transmission name="lin1">
-		<type>transmission_interface/SimpleTransmission</type>
-		<joint name="p1_joint">
-			<hardwareInterface>hardware_interface/EffortJointInterface</hardwareInterface>
-		</joint>
-		<actuator name="lin_motor1">
-			<hardwareInterface>EffortJointInterface</hardwareInterface>
-			<mechanicalReduction>1</mechanicalReduction>
-		</actuator>
-	</transmission>
 	<joint name="p2_joint" type="prismatic">
 		<parent link="p1"/>
@@ -57,23 +48,13 @@
 				xyz="0.0 0.0 0.0"
 				rpy="0.0 0.0 0.0" />
-			<mass value="0.01" />
+			<mass value="0.001" />
 			<inertia
 				ixx="1e-2"
-				ixy="0.0"
-				ixz="0.0"
+				ixy="0.000001"
+				ixz="0.000001"
 				iyy="1e-2"
-				iyz="0.0"
+				iyz="0.000001"
 				izz="1e-2" />
 		</inertial>
-		<surface>
-			<friction>
-				<ode>
-					<mu>0</mu>
-					<mu2>0</mu2>
-					<fdir1>0 1.0 0</fdir1>
-					<implicit_spring_damper>true</implicit_spring_damper>
-				</ode>
-			</friction>
-		</surface>
 	</link>
 	<gazebo reference="p2">
@@ -81,32 +62,20 @@
 		<mu2>0</mu2>
 	</gazebo>
-	<transmission name="lin2">
-		<type>transmission_interface/SimpleTransmission</type>
-		<joint name="p2_joint">
-			<hardwareInterface>hardware_interface/EffortJointInterface</hardwareInterface>
-		</joint>
-		<actuator name="lin_motor2">
-			<hardwareInterface>EffortJointInterface</hardwareInterface>
-			<mechanicalReduction>1</mechanicalReduction>
-		</actuator>
-	</transmission>
-  <joint name="fixed_joint" type="fixed">
-    <parent link="p2"/>
-    <origin link="base_link"/>
-  </joint> -->
-  <joint name="base_joint" type="planar">
-    <origin xyz = "5 0 0" rpy="0 0 0"/>
-    <parent link="world"/>
-    <child link="base_link"/>
-  </joint>
+	<joint name="r_joint" type="continuous">
+		<axis xyz="0 0 1"/>
+		<parent link="p2"/>
+		<origin rpy="0 0 0" xyz="0 0 0"/>
+		<child link="base_link"/>
+		<dynamics damping="0.0" friction="0.0"/>
+	</joint>
   <link name="base_link">
-    <visual>
-      <geometry>
-        <box size="0.09 0.09 0.09"/>
-      </geometry>
-      <origin xyz="0.045 0 0" rpy="0 0 0" />
-      <material name="blue">
-        <color rgba="0 0 .8 1"/>
-      </material>
+	<visual>
+    	<geometry>
+        	<box size="0.09 0.09 0.09"/>
+      	</geometry>
+      	<origin xyz="0.045 0 0" rpy="0 0 0" />
+      	<material name="blue">
+       		<color rgba="0 0 .8 1"/>
+      	</material>
     </visual>
     <collision>
@@ -123,33 +92,8 @@
   </link>
   <gazebo reference="base_link">
-      <mu1>0</mu1>
-      <mu2>0</mu2>
+	<mu1>0</mu1>
+    <mu2>0</mu2>
+	<kp>1000000</kp>
+	<kd>0</kd>
   </gazebo>
-<!--
-  <link name="ring_link">
-    <visual>
-      <geometry>
-        <cylinder length="0.01" radius="0.1"/>
-      </geometry>
-       //htan se sxolio afto<origin xyz="0 0 0.525" />
-      <material name="blue">
-        <color rgba="0 0 .8 1"/>
-      </material>
-    </visual>
-    <collision>
-      <geometry>
-        <cylinder length="0.01" radius="0.1"/>
-      </geometry>
-    </collision>
-    <inertial>
-      <mass value="1"/>
-      <inertia ixx="0.04" ixy="0.0" ixz="0.0" iyy="0.4" iyz="0.0" izz="0.02"/>
-    </inertial>
-  </link>
--->
-  <!-- <joint name="simple_joint" type="continuous">
-    <parent link="base_link"/>
-    <child link="ring_link"/>
-    //htan se sxolio afto <origin xyz="0 0 0.5" />
-  </joint> -->
 </robot>
