Commit message: paei kala to robot kounietai

File: src/cepheus_description/urdf/cepheus.xacro (robot description, xacro)
@@ -123,5 +123,5 @@
 				xyz="0.0024 0.02937 0.15711"
 				rpy="0 0 0" />
-			<mass value="13.3" />
+			<mass value="400" />
 			<inertia
 				ixx="0"
@@ -130,5 +130,5 @@
 				iyy="0"
 				iyz="0"
-				izz="0.160875" />
+				izz="200" />
 		</inertial>
 		<visual>
@@ -214,5 +214,5 @@
 				xyz="0.119 0 0"
 				rpy="0 0 0" />
-			<mass value="0.083" />
+			<mass value="50" />
 			<inertia
 				ixx="0"
@@ -221,5 +221,5 @@
 				iyy="0"
 				iyz="0"
-				izz="0.000346" />
+				izz="16.67" />
 		</inertial>
 		<visual>
@@ -272,5 +272,5 @@
 				xyz="0.119 0 0"
 				rpy="0 0 0" />
-			<mass value="0.187" />
+			<mass value="50" />
 			<inertia
 				ixx="0"
@@ -279,5 +279,5 @@
 				iyy="0"
 				iyz="0"
-				izz="0.000346" />
+				izz="16.67" />
 		</inertial>
 		<visual>
@@ -330,5 +330,5 @@
 				xyz="0.01947 -0.00226 -0.00228"
 				rpy="0 0 0" />
-			<mass value="0.03547" />
+			<mass value="50" />
 			<inertia
 				ixx="0.0926325136613974"
@@ -337,5 +337,5 @@
 				iyy="0.0752633235560557"
 				iyz="0.00191940596202769"
-				izz="0.0919273463968869" />
+				izz="4.17" />
 		</inertial>
 		<visual>

File: src/cepheus_description/urdf/simple_ring.xacro (robot description, xacro)
@@ -24,5 +24,5 @@
     </collision>
     <inertial>
-      <mass value="1.0"/>
+      <mass value="90.0"/>
       <inertia ixx="0.0833" ixy="0" ixz="0" iyy="0.0833" iyz="0" izz="0.0833"/>
     </inertial>

Commit message: prismatic X done, need to add dummy link and prismatic Y

File: src/cepheus_description/urdf/cepheus.xacro (robot description, xacro)
@@ -118,5 +118,50 @@
 	den ksero ti kanoun akomh, nikiforos -->
 	<!-- extra links addition END -->
-	<link name="cepheus">
+	<link name="world">
+		<inertial>
+			<origin
+				xyz="0.00 0.0 0.0"
+				rpy="0 0 0" />
+			<mass value="10000" />
+			<inertia
+				ixx="0"
+				ixy="0"
+				ixz="0"
+				iyy="0"
+				iyz="0"
+				izz="1000" />
+		</inertial>
+		<visual>
+			<material name="LightGrey"/>
+			<geometry>
+				<box size="1000 1000 0.001"/>
+			</geometry>
+		</visual>
+		<collision>
+			<origin
+				xyz="0 0 0"
+				rpy="0 0 0" />
+			<geometry>
+				<box size="1000 1000 0.001"/>
+			</geometry>
+		</collision>
+	</link>
+	<joint name="thrusterx_joint" type="prismatic">
+		<parent link="world"/>
+		<child link="cepheus_base"/>
+		<origin xyz="0 0 0" rpy="0 0 0"/>
+		<axis xyz="1 0 0"/>
+		<limit lower="-100.0" upper="100.0" effort="10.0" velocity="1.0"/>
+		<dynamics damping="1.0" friction="1.0"/>
+	</joint>
+	<!-- <joint name="thrustery_joint" type="prismatic">
+		<parent link="world"/>
+		<child link="cepheus_base"/>
+		<origin xyz="0 0 0" rpy="0 0 0"/>
+		<axis xyz="0 1 0"/>
+		<limit lower="-100.0" upper="100.0" effort="10.0" velocity="1.0"/>
+		<dynamics damping="1.0" friction="1.0"/>
+	</joint> -->
+	<link name="cepheus_base">
 		<inertial>
 			<origin
@@ -150,6 +195,28 @@
 		</collision>
 	</link>
+	<transmission name="tran0x">
+		<type>
+			transmission_interface/SimpleTransmission</type>
+		<joint name="thrusterx_joint">
+			<hardwareInterface>hardware_interface/EffortJointInterface</hardwareInterface>
+		</joint>
+		<actuator name="motor0x">
+			<hardwareInterface>EffortJointInterface</hardwareInterface>
+			<mechanicalReduction>1</mechanicalReduction>
+		</actuator>
+	</transmission>
+	<!-- <transmission name="tran0y">
+		<type>
+			transmission_interface/SimpleTransmission</type>
+		<joint name="thrustery_joint">
+			<hardwareInterface>hardware_interface/EffortJointInterface</hardwareInterface>
+		</joint>
+		<actuator name="motor0y">
+			<hardwareInterface>EffortJointInterface</hardwareInterface>
+			<mechanicalReduction>1</mechanicalReduction>
+		</actuator>
+	</transmission> -->
 	<joint name="reaction_wheel_joint" type="continuous">
-		<parent link="cepheus"/>
+		<parent link="cepheus_base"/>
 		<child link="reaction_wheel"/>
 		<origin xyz="0.065 0 0.03815" rpy="0 0 0"/>
@@ -178,5 +245,5 @@
 		</inertial>
 	</link>
-	<gazebo reference="cepheus">
+	<gazebo reference="cepheus_base">
 		<mu1>0</mu1>
 		<mu2>0</mu2>
@@ -193,9 +260,9 @@
 		</actuator>
 	</transmission>
-	<joint name="left_shoulder" type="revolute">
+	<joint name="left_shoulder_joint" type="revolute">
 		<origin
 			xyz="0.17271 0.091404 0.05875"
 			rpy="0 0 0" />
-		<parent link="cepheus" />
+		<parent link="cepheus_base" />
 		<child link="left_arm" />
 		<axis xyz="0 0 1" />
@@ -243,5 +310,5 @@
 	<transmission name="tran2">
 		<type>transmission_interface/SimpleTransmission</type>
-		<joint name="left_shoulder">
+		<joint name="left_shoulder_joint">
 			<hardwareInterface>hardware_interface/EffortJointInterface</hardwareInterface>
 		</joint>
@@ -251,5 +318,5 @@
 		</actuator>
 	</transmission>
-	<joint name="left_elbow" type="revolute">
+	<joint name="left_elbow_joint" type="revolute">
 		<origin
 			xyz="0.1810 0 0"
@@ -301,5 +368,5 @@
 	<transmission name="tran3">
 		<type>transmission_interface/SimpleTransmission</type>
-		<joint name="left_elbow">
+		<joint name="left_elbow_joint">
 			<hardwareInterface>hardware_interface/EffortJointInterface</hardwareInterface>
 		</joint>
@@ -309,5 +376,5 @@
 		</actuator>
 	</transmission>
-	<joint name="left_wrist" type="revolute">
+	<joint name="left_wrist_joint" type="revolute">
 		<origin
 			xyz="0.15965 0.01176 -0.00838"
@@ -359,5 +426,5 @@
 	<transmission name="tran4">
 		<type>transmission_interface/SimpleTransmission</type>
-		<joint name="left_wrist">
+		<joint name="left_wrist_joint">
 			<hardwareInterface>hardware_interface/EffortJointInterface</hardwareInterface>
 		</joint>
@@ -394,6 +461,6 @@
 		</inertial>
 	</link> -->
-	<!-- <gazebo reference="left_wrist">
-		<sensor name="left_wrist_force_torque" type="force_torque">
+	<!-- <gazebo reference="left_wrist_joint">
+		<sensor name="left_wrist_joint_force_torque" type="force_torque">
     	<always_on>true</always_on>
     	<update_rate>20.0</update_rate>
@@ -412,9 +479,9 @@
 			<topicName>ft_sensor_topic</topicName>
 			<gaussianNoise>0.0</gaussianNoise>
-			<jointName>left_wrist</jointName>
+			<jointName>left_wrist_joint</jointName>
 			<visualize>true</visualize>
 		</plugin>
 	</gazebo> -->
-	<gazebo reference="left_wrist">
+	<gazebo reference="left_wrist_joint">
 		<disableFixedJointLumping>true</disableFixedJointLumping>
 		<sensor name="my_cool_sensor" type="force_torque">
@@ -429,5 +496,5 @@
 			<updateRate>0</updateRate>   <!--poly shmantiko na einai 0, allios kanei bug!!!!(nikhforos)-->
 			<topicName>ft_sensor_topic</topicName>
-			<jointName>left_wrist</jointName>
+			<jointName>left_wrist_joint</jointName>
 		</plugin>
 	</gazebo>

Commit message: doulevei to robot alla kanei treles

File: src/cepheus_description/urdf/cepheus.xacro (robot description, xacro)
@@ -21,6 +21,6 @@
 		<dynamics damping="0" friction="0"/>
 	</joint> -->
-	<!--
-	<joint name="p1_joint" type="prismatic">
+	<link name = "world"/>
+	<joint name="thrusterx_joint" type="prismatic">
 		<parent link="world"/>
 		<child link="p1"/>
@@ -50,5 +50,5 @@
 	<transmission name="lin1">
 		<type>transmission_interface/SimpleTransmission</type>
-		<joint name="p1_joint">
+		<joint name="thrusterx_joint">
 			<hardwareInterface>hardware_interface/EffortJointInterface</hardwareInterface>
 		</joint>
@@ -58,7 +58,7 @@
 		</actuator>
 	</transmission>
-	<joint name="p2_joint" type="prismatic">
+	<joint name="thrustery_joint" type="prismatic">
 		<parent link="p1"/>
-		<child link="p2"/>
+		<child link="cepheus_base"/>
 		<axis xyz="0 1 0"/>
 		<limit
@@ -71,5 +71,5 @@
 			friction="0"/>
 	</joint>
-	<link name="p2">
+	<!-- <link name="p2">
 		<inertial>
 			<origin
@@ -99,8 +99,8 @@
 		<mu1>0</mu1>
 		<mu2>0</mu2>
-	</gazebo>
+	</gazebo> -->
 	<transmission name="lin2">
 		<type>transmission_interface/SimpleTransmission</type>
-		<joint name="p2_joint">
+		<joint name="thrustery_joint">
 			<hardwareInterface>hardware_interface/EffortJointInterface</hardwareInterface>
 		</joint>
@@ -110,13 +110,16 @@
 		</actuator>
 	</transmission>
-	<joint name="r_joint" type="continuous">
+	<!-- <joint name="p2_to_base" type="fixed">
+		<parent link ="p2"/>
+		<child link="cepheus_base"/>
+	</joint> -->
+	<!-- <joint name="r_joint" type="continuous">
 		<axis xyz="0 0 1"/>
 		<parent link="p2"/>
 		<origin rpy="0 0 0" xyz="0 0 0"/>
 		<child link="cepheus"/>
-	</joint>
-	den ksero ti kanoun akomh, nikiforos -->
+	</joint> -->
 	<!-- extra links addition END -->
-	<link name="world">
+	<!-- <link name="world">
 		<inertial>
 			<origin
@@ -146,17 +149,46 @@
 			</geometry>
 		</collision>
-	</link>
-	<joint name="thrusterx_joint" type="prismatic">
+	</link> -->
+	<!-- <joint name="thrusterx_joint" type="prismatic">
 		<parent link="world"/>
-		<child link="cepheus_base"/>
-		<origin xyz="0 0 0" rpy="0 0 0"/>
+		<child link="dummy_link"/>
+		<origin xyz="0 0 0"/>
 		<axis xyz="1 0 0"/>
 		<limit lower="-100.0" upper="100.0" effort="10.0" velocity="1.0"/>
-		<dynamics damping="1.0" friction="1.0"/>
-	</joint>
-	<!-- <joint name="thrustery_joint" type="prismatic">
-		<parent link="world"/>
+		<dynamics damping="1.0" />
+	</joint>
+		<link name="dummy_link">
+		<inertial>
+			<origin
+				xyz="0.0 0.0 0.0"
+				rpy="0 0 0" />
+			<mass value="1" />
+			<inertia
+				ixx="0"
+				ixy="0"
+				ixz="0"
+				iyy="0"
+				iyz="0"
+				izz="0.001" />
+		</inertial>
+		<visual>
+			<material name="LightGrey"/>
+			<geometry>
+				<box size="0.001 0.001 0.001"/>
+			</geometry>
+		</visual>
+		<collision>
+			<origin
+				xyz="0 0 0"
+				rpy="0 0 0" />
+			<geometry>
+				<box size="0.001 0.001 0.001"/>
+			</geometry>
+		</collision>
+	</link>
+	<joint name="thrustery_joint" type="prismatic">
+		<parent link="dummy_link"/>
 		<child link="cepheus_base"/>
-		<origin xyz="0 0 0" rpy="0 0 0"/>
+		<origin xyz="0 0 0"/>
 		<axis xyz="0 1 0"/>
 		<limit lower="-100.0" upper="100.0" effort="10.0" velocity="1.0"/>
@@ -195,5 +227,5 @@
 		</collision>
 	</link>
-	<transmission name="tran0x">
+	<!-- <transmission name="tran0x">
 		<type>
 			transmission_interface/SimpleTransmission</type>
@@ -206,5 +238,5 @@
 		</actuator>
 	</transmission>
-	<!-- <transmission name="tran0y">
+	<transmission name="tran0y">
 		<type>
 			transmission_interface/SimpleTransmission</type>

Commit message: eftiaksa to base force plugin alla mou kanoun kolpa ta joints

File: src/cepheus_description/urdf/cepheus.xacro (robot description, xacro)
@@ -21,5 +21,5 @@
 		<dynamics damping="0" friction="0"/>
 	</joint> -->
-	<link name = "world"/>
+	<!-- <link name = "world"/>
 	<joint name="thrusterx_joint" type="prismatic">
 		<parent link="world"/>
@@ -70,5 +70,5 @@
 			damping="0"
 			friction="0"/>
-	</joint>
+	</joint> -->
 	<!-- <link name="p2">
 		<inertial>
@@ -100,5 +100,5 @@
 		<mu2>0</mu2>
 	</gazebo> -->
-	<transmission name="lin2">
+	<!-- <transmission name="lin2">
 		<type>transmission_interface/SimpleTransmission</type>
 		<joint name="thrustery_joint">
@@ -109,5 +109,5 @@
 			<mechanicalReduction>1</mechanicalReduction>
 		</actuator>
-	</transmission>
+	</transmission> -->
 	<!-- <joint name="p2_to_base" type="fixed">
 		<parent link ="p2"/>
@@ -531,3 +531,12 @@
 		</plugin>
 	</gazebo>
+	<gazebo>
+		<plugin filename="libgazebo_ros_force.so" name="gazebo_ros_force" >
+			<!-- <alwaysOn>true</alwaysOn> -->
+			<!-- <update>100</update> -->
+			<!-- <updateRate>0</updateRate> anti gia 100 -->
+			<bodyName>cepheus_base</bodyName>
+			<topicName>force_base_topic</topicName>
+		</plugin>
+	</gazebo>
 </robot>

Commit message: allaksa inertias, evala 3 joints san odhgous, psilodoulevei

File: src/cepheus_description/urdf/cepheus.xacro (robot description, xacro)
@@ -4,23 +4,7 @@
 	<xacro:include filename="$(find cepheus_description)/urdf/materials.xacro" />
 	<xacro:property name="camera_link" value="0.05" /> <!-- Size of square 'camera' box -->
-	<!--<link name="world">
-		<joint name="world_joint" type="continuous">
-			<axis xyz="0 0 1"/>
-			<parent link="world"/>
-			<origin rpy="0 0 0" xyz="0 0 0"/>
-			<child link="cepheus"/>
-			<dynamics damping="0" friction="0"/>
-		</joint>
-	</link>-->
-	<!-- extra links addition START -->
-	<!-- <joint name="world_joint" type="continuous">
-		<axis xyz="0 0 1"/>
-		<parent link="world"/>
-		<origin rpy="0 0 0" xyz="0 0 0"/>
-		<child link="cepheus"/>
-		<dynamics damping="0" friction="0"/>
-	</joint> -->
-	<!-- <link name = "world"/>
-	<joint name="thrusterx_joint" type="prismatic">
+	<link name="world"/>
+<!-- thanks pelekoudas -->
+	<joint name="p1_joint" type="prismatic">
 		<parent link="world"/>
 		<child link="p1"/>
@@ -50,5 +34,5 @@
 	<transmission name="lin1">
 		<type>transmission_interface/SimpleTransmission</type>
-		<joint name="thrusterx_joint">
+		<joint name="p1_joint">
 			<hardwareInterface>hardware_interface/EffortJointInterface</hardwareInterface>
 		</joint>
@@ -58,7 +42,7 @@
 		</actuator>
 	</transmission>
-	<joint name="thrustery_joint" type="prismatic">
+	<joint name="p2_joint" type="prismatic">
 		<parent link="p1"/>
-		<child link="cepheus_base"/>
+		<child link="p2"/>
 		<axis xyz="0 1 0"/>
 		<limit
@@ -70,6 +54,6 @@
 			damping="0"
 			friction="0"/>
-	</joint> -->
-	<!-- <link name="p2">
+	</joint>
+	<link name="p2">
 		<inertial>
 			<origin
@@ -99,8 +83,8 @@
 		<mu1>0</mu1>
 		<mu2>0</mu2>
-	</gazebo> -->
-	<!-- <transmission name="lin2">
-		<type>transmission_interface/SimpleTransmission</type>
-		<joint name="thrustery_joint">
+	</gazebo>
+	<transmission name="lin2">
+		<type>transmission_interface/SimpleTransmission</type>
+		<joint name="p2_joint">
 			<hardwareInterface>hardware_interface/EffortJointInterface</hardwareInterface>
 		</joint>
@@ -109,144 +93,43 @@
 			<mechanicalReduction>1</mechanicalReduction>
 		</actuator>
-	</transmission> -->
-	<!-- <joint name="p2_to_base" type="fixed">
-		<parent link ="p2"/>
-		<child link="cepheus_base"/>
-	</joint> -->
-	<!-- <joint name="r_joint" type="continuous">
+	</transmission>
+	<joint name="r_joint" type="continuous">
 		<axis xyz="0 0 1"/>
 		<parent link="p2"/>
 		<origin rpy="0 0 0" xyz="0 0 0"/>
-		<child link="cepheus"/>
-	</joint> -->
-	<!-- extra links addition END -->
-	<!-- <link name="world">
-		<inertial>
-			<origin
-				xyz="0.00 0.0 0.0"
-				rpy="0 0 0" />
-			<mass value="10000" />
-			<inertia
-				ixx="0"
-				ixy="0"
-				ixz="0"
-				iyy="0"
-				iyz="0"
-				izz="1000" />
-		</inertial>
-		<visual>
+		<child link="cepheus_base"/>
+	</joint>
+	<link name="cepheus_base">
+		<inertial>
+			<origin
+				xyz="0.0024 0.02937 0.15711"
+				rpy="0 0 0" />
+			<mass value="13.3" />
+			<inertia
+				ixx="0"
+				ixy="0"
+				ixz="0"
+				iyy="0"
+				iyz="0"
+				izz="0.160875" />
+		</inertial>
+		<visual>
+			<origin
+				xyz="0 0 0"
+				rpy="0 0 0" />
+			<geometry>
+				<mesh filename="package://cepheus_description/urdf/meshes/cepheus.STL" />
+			</geometry>
 			<material name="LightGrey"/>
-			<geometry>
-				<box size="1000 1000 0.001"/>
-			</geometry>
 		</visual>
 		<collision>
 			<origin
-				xyz="0 0 0"
-				rpy="0 0 0" />
-			<geometry>
-				<box size="1000 1000 0.001"/>
+				xyz="0 0 0.215"
+				rpy="0 0 0" />
+			<geometry>
+				<cylinder length="0.43" radius="0.2"/>
 			</geometry>
 		</collision>
-	</link> -->
-	<!-- <joint name="thrusterx_joint" type="prismatic">
-		<parent link="world"/>
-		<child link="dummy_link"/>
-		<origin xyz="0 0 0"/>
-		<axis xyz="1 0 0"/>
-		<limit lower="-100.0" upper="100.0" effort="10.0" velocity="1.0"/>
-		<dynamics damping="1.0" />
-	</joint>
-		<link name="dummy_link">
-		<inertial>
-			<origin
-				xyz="0.0 0.0 0.0"
-				rpy="0 0 0" />
-			<mass value="1" />
-			<inertia
-				ixx="0"
-				ixy="0"
-				ixz="0"
-				iyy="0"
-				iyz="0"
-				izz="0.001" />
-		</inertial>
-		<visual>
-			<material name="LightGrey"/>
-			<geometry>
-				<box size="0.001 0.001 0.001"/>
-			</geometry>
-		</visual>
-		<collision>
-			<origin
-				xyz="0 0 0"
-				rpy="0 0 0" />
-			<geometry>
-				<box size="0.001 0.001 0.001"/>
-			</geometry>
-		</collision>
-	</link>
-	<joint name="thrustery_joint" type="prismatic">
-		<parent link="dummy_link"/>
-		<child link="cepheus_base"/>
-		<origin xyz="0 0 0"/>
-		<axis xyz="0 1 0"/>
-		<limit lower="-100.0" upper="100.0" effort="10.0" velocity="1.0"/>
-		<dynamics damping="1.0" friction="1.0"/>
-	</joint> -->
-	<link name="cepheus_base">
-		<inertial>
-			<origin
-				xyz="0.0024 0.02937 0.15711"
-				rpy="0 0 0" />
-			<mass value="400" />
-			<inertia
-				ixx="0"
-				ixy="0"
-				ixz="0"
-				iyy="0"
-				iyz="0"
-				izz="200" />
-		</inertial>
-		<visual>
-			<origin
-				xyz="0 0 0"
-				rpy="0 0 0" />
-			<geometry>
-				<mesh filename="package://cepheus_description/urdf/meshes/cepheus.STL" />
-			</geometry>
-			<material name="LightGrey"/>
-		</visual>
-		<collision>
-			<origin
-				xyz="0 0 0.215"
-				rpy="0 0 0" />
-			<geometry>
-				<cylinder length="0.43" radius="0.2"/>
-			</geometry>
-		</collision>
-	</link>
-	<!-- <transmission name="tran0x">
-		<type>
-			transmission_interface/SimpleTransmission</type>
-		<joint name="thrusterx_joint">
-			<hardwareInterface>hardware_interface/EffortJointInterface</hardwareInterface>
-		</joint>
-		<actuator name="motor0x">
-			<hardwareInterface>EffortJointInterface</hardwareInterface>
-			<mechanicalReduction>1</mechanicalReduction>
-		</actuator>
-	</transmission>
-	<transmission name="tran0y">
-		<type>
-			transmission_interface/SimpleTransmission</type>
-		<joint name="thrustery_joint">
-			<hardwareInterface>hardware_interface/EffortJointInterface</hardwareInterface>
-		</joint>
-		<actuator name="motor0y">
-			<hardwareInterface>EffortJointInterface</hardwareInterface>
-			<mechanicalReduction>1</mechanicalReduction>
-		</actuator>
-	</transmission> -->
+	</link>
 	<joint name="reaction_wheel_joint" type="continuous">
 		<parent link="cepheus_base"/>
@@ -313,12 +196,12 @@
 				xyz="0.119 0 0"
 				rpy="0 0 0" />
-			<mass value="50" />
-			<inertia
-				ixx="0"
-				ixy="0"
-				ixz="0"
-				iyy="0"
-				iyz="0"
-				izz="16.67" />
+			<mass value="0.083" />
+			<inertia
+				ixx="0"
+				ixy="0"
+				ixz="0"
+				iyy="0"
+				iyz="0"
+				izz="0.000346" />
 		</inertial>
 		<visual>
@@ -371,12 +254,12 @@
 				xyz="0.119 0 0"
 				rpy="0 0 0" />
-			<mass value="50" />
-			<inertia
-				ixx="0"
-				ixy="0"
-				ixz="0"
-				iyy="0"
-				iyz="0"
-				izz="16.67" />
+			<mass value="0.187" />
+			<inertia
+				ixx="0"
+				ixy="0"
+				ixz="0"
+				iyy="0"
+				iyz="0"
+				izz="0.000346" />
 		</inertial>
 		<visual>
@@ -429,12 +312,12 @@
 				xyz="0.01947 -0.00226 -0.00228"
 				rpy="0 0 0" />
-			<mass value="50" />
-			<inertia
-				ixx="0.0926325136613974"
-				ixy="-0.00333421740190982"
-				ixz="0.00529966557344093"
-				iyy="0.0752633235560557"
-				iyz="0.00191940596202769"
-				izz="4.17" />
+			<mass value="0.03547" />
+			<inertia
+				ixx="0"
+				ixy="0"
+				ixz="0"
+				iyy="0"
+				iyz="0"
+				izz="0.0919273463968869" />
 		</inertial>
 		<visual>
@@ -466,31 +349,4 @@
 		</actuator>
 	</transmission>
-	<!-- <joint name="camera_joint" type="fixed">
-		<axis xyz="0 1 0" />
-		<origin xyz="0 0 3.0" rpy="0 1.5708 1.5708"/>
-		<parent link="world"/>
-		<child link="camera_link"/>
-	</joint> -->
-	<!-- Camera -->
-	<!-- <link name="camera_link">
-		<collision>
-			<origin xyz="0 0 0" rpy="0 0 0"/>
-			<geometry>
-				<box size="${camera_link} ${camera_link} ${camera_link}"/>
-			</geometry>
-		</collision>
-		<visual>
-			<origin xyz="0 0 0" rpy="0 0 0"/>
-			<geometry>
-				<box size="${camera_link} ${camera_link} ${camera_link}"/>
-			</geometry>
-			<material name="red"/>
-		</visual>
-		<inertial>
-			<mass value="1e-5" />
-			<origin xyz="0 0 0" rpy="0 0 0"/>
-			<inertia ixx="1e-6" ixy="0" ixz="0" iyy="1e-6" iyz="0" izz="1e-6" />
-		</inertial>
-	</link> -->
 	<!-- <gazebo reference="left_wrist_joint">
 		<sensor name="left_wrist_joint_force_torque" type="force_torque">

File: src/cepheus_description/urdf/simple_ring.xacro (robot description, xacro)
@@ -24,6 +24,6 @@
     </collision>
     <inertial>
-      <mass value="90.0"/>
-      <inertia ixx="0.0833" ixy="0" ixz="0" iyy="0.0833" iyz="0" izz="0.0833"/>
+      <mass value="9.0"/>
+      <inertia ixx="0.00833" ixy="0" ixz="0" iyy="0.00833" iyz="0" izz="0.00833"/>
     </inertial>
   </link>
@@ -44,6 +44,6 @@
     </collision>
     <inertial>
-      <mass value="10"/>
-      <inertia ixx="0.4" ixy="0.0" ixz="0.0" iyy="0.4" iyz="0.0" izz="0.2"/>
+      <mass value="1"/>
+      <inertia ixx="0.04" ixy="0.0" ixz="0.0" iyy="0.4" iyz="0.0" izz="0.02"/>
     </inertial>
   </link>
