Commit message: eftiaksa xd, na allakso xacro

File: src/cepheus_description/urdf/cepheus.xacro (robot description, xacro)
@@ -105,12 +105,12 @@
 				xyz="0.0024 0.02937 0.15711"
 				rpy="0 0 0" />
-			<mass value="13.3" />
-			<inertia
-				ixx="0"
-				ixy="0"
-				ixz="0"
-				iyy="0"
-				iyz="0"
-				izz="0.160875" /> <!-- 13.3 -->
+			<mass value="53.53" />
+			<inertia
+				ixx="0.0001"
+				ixy="0.0001"
+				ixz="0.0001"
+				iyy="0.0001"
+				iyz="0.0001"
+				izz="2.2491" /> <!-- 13.3 -->
 		</inertial>
 		<visual>
@@ -196,12 +196,12 @@
 				xyz="0.119 0 0"
 				rpy="0 0 0" />
-			<mass value="0.083" />
-			<inertia
-				ixx="0"
-				ixy="0"
-				ixz="0"
-				iyy="0"
-				iyz="0"
-				izz="0.000346" /> <!--0.0083 -->
+			<mass value="0.4409" />
+			<inertia
+				ixx="0.0001"
+				ixy="0.0001"
+				ixz="0.0001"
+				iyy="0.0001"
+				iyz="0.0001"
+				izz="0.0068" /> <!--0.0083 -->
 		</inertial>
 		<visual>
@@ -210,5 +210,6 @@
 				rpy="0 0 0" />
 			<geometry>
-				<mesh filename="package://cepheus_description/urdf/meshes/left_arm.STL" />
+				<!-- <mesh filename="package://cepheus_description/urdf/meshes/left_arm.STL" /> -->
+				<box size="0.37 0.02 0.02"/>
 			</geometry>
 			<material name="LightGrey"/>
@@ -219,5 +220,5 @@
 				rpy="0 0 0" />
 			<geometry>
-				<box size="0.13 0.02 0.02"/>
+				<box size="0.37 0.02 0.02"/>
 			</geometry>
 		</collision>
@@ -234,7 +235,7 @@
 	</transmission>
 	<joint name="left_elbow_joint" type="revolute">
-		<origin
+		<!-- <origin
 			xyz="0.1810 0 0"
-			rpy="0 0 0" />
+			rpy="0 0 0" /> -->
 		<parent link="left_arm" />
 		<child link="left_forearm" />
@@ -251,15 +252,15 @@
 	<link name="left_forearm">
 		<inertial>
-			<origin
+			<!-- <origin
 				xyz="0.119 0 0"
-				rpy="0 0 0" />
-			<mass value="0.187" />
-			<inertia
-				ixx="0"
-				ixy="0"
-				ixz="0"
-				iyy="0"
-				iyz="0"
-				izz="0.000346" /> <!--0.0199 -->
+				rpy="0 0 0" /> -->
+			<mass value="0.1304" />
+			<inertia
+				ixx="0.0001"
+				ixy="0.0001"
+				ixz="0.0001"
+				iyy="0.0001"
+				iyz="0.0001"
+				izz="0.0010" /> <!--0.0199 -->
 		</inertial>
 		<visual>
@@ -268,5 +269,6 @@
 				rpy="0 0 0" />
 			<geometry>
-				<mesh filename="package://cepheus_description/urdf/meshes/left_forearm.STL" />
+				<!-- <mesh filename="package://cepheus_description/urdf/meshes/left_forearm.STL" /> -->
+				<box size="0.286 0.025 0.025"/>
 			</geometry>
 			<material name="LightGrey"/>
@@ -277,5 +279,5 @@
 				rpy="0 0 0" />
 			<geometry>
-				<box size="0.13 0.025 0.025"/>
+				<box size="0.286 0.025 0.025"/>
 			</geometry>
 		</collision>
@@ -292,7 +294,7 @@
 	</transmission>
 	<joint name="left_wrist_joint" type="revolute">
-		<origin
+		<!-- <origin
 			xyz="0.15965 0.01176 -0.00838"
-			rpy="0 0 0 " />
+			rpy="0 0 0 " /> -->
 		<parent link="left_forearm" />
 		<child link="left_grip" />
@@ -309,15 +311,15 @@
 	<link name="left_grip">
 		<inertial>
-			<origin
+			<!-- <origin
 				xyz="0.01947 -0.00226 -0.00228"
-				rpy="0 0 0" />
-			<mass value="0.03547" />
-			<inertia
-				ixx="0"
-				ixy="0"
-				ixz="0"
-				iyy="0"
-				iyz="0"
-				izz="0.091927" /> <!--0.00101 "-->
+				rpy="0 0 0" /> -->
+			<mass value="6.2229" />
+			<inertia
+				ixx="0.0001"
+				ixy="0.0001"
+				ixz="0.0001"
+				iyy="0.0001"
+				iyz="0.0001"
+				izz="0.0787" /> <!--0.00101 "-->
 		</inertial>
 		<visual>
@@ -394,4 +396,5 @@
 			<bodyName>cepheus_base</bodyName>
 			<topicName>force_base_topic</topicName>
+			<force_reference_frame>world</force_reference_frame>
 		</plugin>
 	</gazebo>

Commit message: vaggelis me eftiakse cap

File: src/cepheus_description/urdf/cepheus.xacro (robot description, xacro)
@@ -193,7 +193,8 @@
 	<link name="left_arm">
 		<inertial>
-			<origin
+			<!-- <origin
 				xyz="0.119 0 0"
-				rpy="0 0 0" />
+				rpy="0 0 0" /> -->
+			<origin xyz="0.185 0 0" rpy="0 0 0"/>
 			<mass value="0.4409" />
 			<inertia
@@ -206,7 +207,8 @@
 		</inertial>
 		<visual>
-			<origin
+			<!-- <origin
 				xyz="0 -0.0085 0"
-				rpy="0 0 0" />
+				rpy="0 0 0" /> -->
+			<origin xyz="0.185 0 0" rpy="0 0 0"/>
 			<geometry>
 				<!-- <mesh filename="package://cepheus_description/urdf/meshes/left_arm.STL" /> -->
@@ -216,7 +218,8 @@
 		</visual>
 		<collision>
-			<origin
+			<!-- <origin
 				xyz="0.08 0.0 0.01"
-				rpy="0 0 0" />
+				rpy="0 0 0" /> -->
+			<origin xyz="0.185 0 0" rpy="0 0 0"/>
 			<geometry>
 				<box size="0.37 0.02 0.02"/>
@@ -238,4 +241,5 @@
 			xyz="0.1810 0 0"
 			rpy="0 0 0" /> -->
+		<origin xyz = "0.37 0 0" rpy="0 0 0"/>
 		<parent link="left_arm" />
 		<child link="left_forearm" />
@@ -255,4 +259,5 @@
 				xyz="0.119 0 0"
 				rpy="0 0 0" /> -->
+			<origin xyz="0.143 0 0" rpy="0 0 0"/>
 			<mass value="0.1304" />
 			<inertia
@@ -265,7 +270,8 @@
 		</inertial>
 		<visual>
-			<origin
+			<!-- <origin
 				xyz="0 0 0"
-				rpy="0 0 0" />
+				rpy="0 0 0" /> -->
+			<origin xyz="0.143 0 0" rpy="0 0 0"/>
 			<geometry>
 				<!-- <mesh filename="package://cepheus_description/urdf/meshes/left_forearm.STL" /> -->
@@ -275,7 +281,8 @@
 		</visual>
 		<collision>
-			<origin
+			<!-- <origin
 				xyz="0.105 0.0115 0.0125"
-				rpy="0 0 0" />
+				rpy="0 0 0" /> -->
+			<origin xyz="0.143 0 0" rpy="0 0 0"/>
 			<geometry>
 				<box size="0.286 0.025 0.025"/>
@@ -297,4 +304,5 @@
 			xyz="0.15965 0.01176 -0.00838"
 			rpy="0 0 0 " /> -->
+		<origin xyz="0.286 0 0" rpy="0 0 0"/>
 		<parent link="left_forearm" />
 		<child link="left_grip" />
@@ -324,6 +332,12 @@
 		</inertial>
 		<visual>
-			<origin
-				xyz="0 0 0"
+			<origin xyz="0.036 0 0" rpy="0 0 0"/>
+			<geometry>
+				<box size= "0.072 0.07 0.05" />
+			</geometry>
+		</visual>
+		<visual>
+			<origin
+				xyz="0.072 0 0"
 				rpy="1.5708 0 0"/>
 			<geometry>
@@ -337,5 +351,5 @@
 				rpy="1.5708 0 0" />
 			<geometry>
-				<box size="0.03 0.07 0.05"/>
+				<box size="0.1082 0.07 0.05"/>
 			</geometry>
 		</collision>
@@ -373,5 +387,5 @@
 		</plugin>
 	</gazebo> -->
-	<gazebo reference="left_wrist_joint">
+	<!-- <gazebo reference="left_wrist_joint">
 		<disableFixedJointLumping>true</disableFixedJointLumping>
 		<sensor name="my_cool_sensor" type="force_torque">
@@ -381,4 +395,7 @@
 			</force_torque>
 		</sensor>
+	</gazebo> -->
+	<gazebo reference="left_wrist_joint">
+	<provideFeedback>true</provideFeedback>
 	</gazebo>
 	<gazebo>

Commit message: gyrisa to xacro stou peleq, phra ta r,l,i,m apo afton, leipei r3,l3, to robot kanei KYKLOYS

File: src/cepheus_description/urdf/cepheus.xacro (robot description, xacro)
@@ -4,6 +4,21 @@
 	<xacro:include filename="$(find cepheus_description)/urdf/materials.xacro" />
 	<xacro:property name="camera_link" value="0.05" /> <!-- Size of square 'camera' box -->
-	<link name="world"/>
-<!-- thanks pelekoudas -->
+	<link name="world">
+		<!-- <joint name="world_joint" type="continuous">
+			<axis xyz="0 0 1"/>
+			<parent link="world"/>
+			<origin rpy="0 0 0" xyz="0 0 0"/>
+			<child link="cepheus"/>
+			<dynamics damping="0" friction="0"/>
+		</joint> -->
+	</link>
+	<!-- extra links addition START -->
+	<!-- <joint name="world_joint" type="continuous">
+		<axis xyz="0 0 1"/>
+		<parent link="world"/>
+		<origin rpy="0 0 0" xyz="0 0 0"/>
+		<child link="cepheus"/>
+		<dynamics damping="0" friction="0"/>
+	</joint> -->
 	<joint name="p1_joint" type="prismatic">
 		<parent link="world"/>
@@ -100,4 +115,5 @@
 		<child link="cepheus_base"/>
 	</joint>
+	<!-- extra links addition END -->
 	<link name="cepheus_base">
 		<inertial>
@@ -105,12 +121,12 @@
 				xyz="0.0024 0.02937 0.15711"
 				rpy="0 0 0" />
-			<mass value="53.53" />
-			<inertia
-				ixx="0.0001"
-				ixy="0.0001"
-				ixz="0.0001"
-				iyy="0.0001"
-				iyz="0.0001"
-				izz="2.2491" /> <!-- 13.3 -->
+			<mass value="13.3" />
+			<inertia
+				ixx="0"
+				ixy="0"
+				ixz="0"
+				iyy="0"
+				iyz="0"
+				izz="0.160875" />
 		</inertial>
 		<visual>
@@ -161,8 +177,4 @@
 	</link>
 	<gazebo reference="cepheus_base">
-		<mu1>0</mu1>
-		<mu2>0</mu2>
-	</gazebo>
-	<gazebo reference="reaction_wheel">
 		<mu1>0</mu1>
 		<mu2>0</mu2>
@@ -197,35 +209,31 @@
 	<link name="left_arm">
 		<inertial>
-			<!-- <origin
+			<origin
 				xyz="0.119 0 0"
-				rpy="0 0 0" /> -->
-			<origin xyz="0.185 0 0" rpy="0 0 0"/>
-			<mass value="0.4409" />
-			<inertia
-				ixx="0.0001"
-				ixy="0.0001"
-				ixz="0.0001"
-				iyy="0.0001"
-				iyz="0.0001"
-				izz="0.0068" /> <!--0.0083 -->
-		</inertial>
-		<visual>
-			<!-- <origin
+				rpy="0 0 0" />
+			<mass value="0.083" />
+			<inertia
+				ixx="0"
+				ixy="0"
+				ixz="0"
+				iyy="0"
+				iyz="0"
+				izz="0.000346" />
+		</inertial>
+		<visual>
+			<origin
 				xyz="0 -0.0085 0"
-				rpy="0 0 0" /> -->
-			<origin xyz="0.185 0 0" rpy="0 0 0"/>
-			<geometry>
-				<!-- <mesh filename="package://cepheus_description/urdf/meshes/left_arm.STL" /> -->
-				<box size="0.37 0.02 0.02"/>
+				rpy="0 0 0" />
+			<geometry>
+				<mesh filename="package://cepheus_description/urdf/meshes/left_arm.STL" />
 			</geometry>
 			<material name="LightGrey"/>
 		</visual>
 		<collision>
-			<!-- <origin
+			<origin
 				xyz="0.08 0.0 0.01"
-				rpy="0 0 0" /> -->
-			<origin xyz="0.185 0 0" rpy="0 0 0"/>
-			<geometry>
-				<box size="0.37 0.02 0.02"/>
+				rpy="0 0 0" />
+			<geometry>
+				<box size="0.13 0.02 0.02"/>
 			</geometry>
 		</collision>
@@ -242,8 +250,7 @@
 	</transmission>
 	<joint name="left_elbow_joint" type="revolute">
-		<!-- <origin
+		<origin
 			xyz="0.1810 0 0"
-			rpy="0 0 0" /> -->
-		<origin xyz = "0.37 0 0" rpy="0 0 0"/>
+			rpy="0 0 0" />
 		<parent link="left_arm" />
 		<child link="left_forearm" />
@@ -260,35 +267,31 @@
 	<link name="left_forearm">
 		<inertial>
-			<!-- <origin
+			<origin
 				xyz="0.119 0 0"
-				rpy="0 0 0" /> -->
-			<origin xyz="0.143 0 0" rpy="0 0 0"/>
-			<mass value="0.1304" />
-			<inertia
-				ixx="0.0001"
-				ixy="0.0001"
-				ixz="0.0001"
-				iyy="0.0001"
-				iyz="0.0001"
-				izz="0.0010" /> <!--0.0199 -->
-		</inertial>
-		<visual>
-			<!-- <origin
+				rpy="0 0 0" />
+			<mass value="0.187" />
+			<inertia
+				ixx="0"
+				ixy="0"
+				ixz="0"
+				iyy="0"
+				iyz="0"
+				izz="0.000346" />
+		</inertial>
+		<visual>
+			<origin
 				xyz="0 0 0"
-				rpy="0 0 0" /> -->
-			<origin xyz="0.143 0 0" rpy="0 0 0"/>
-			<geometry>
-				<!-- <mesh filename="package://cepheus_description/urdf/meshes/left_forearm.STL" /> -->
-				<box size="0.286 0.025 0.025"/>
+				rpy="0 0 0" />
+			<geometry>
+				<mesh filename="package://cepheus_description/urdf/meshes/left_forearm.STL" />
 			</geometry>
 			<material name="LightGrey"/>
 		</visual>
 		<collision>
-			<!-- <origin
+			<origin
 				xyz="0.105 0.0115 0.0125"
-				rpy="0 0 0" /> -->
-			<origin xyz="0.143 0 0" rpy="0 0 0"/>
-			<geometry>
-				<box size="0.286 0.025 0.025"/>
+				rpy="0 0 0" />
+			<geometry>
+				<box size="0.13 0.025 0.025"/>
 			</geometry>
 		</collision>
@@ -305,8 +308,7 @@
 	</transmission>
 	<joint name="left_wrist_joint" type="revolute">
-		<!-- <origin
+		<origin
 			xyz="0.15965 0.01176 -0.00838"
-			rpy="0 0 0 " /> -->
-		<origin xyz="0.286 0 0" rpy="0 0 0"/>
+			rpy="0 0 0 " />
 		<parent link="left_forearm" />
 		<child link="left_grip" />
@@ -315,5 +317,5 @@
 			lower="-1.570796327"
 			upper="1.570796327"
-			effort="10"
+			effort="1"
 			velocity="10" />
 		<dynamics
@@ -323,26 +325,20 @@
 	<link name="left_grip">
 		<inertial>
-			<!-- <origin
+			<origin
 				xyz="0.01947 -0.00226 -0.00228"
-				rpy="0 0 0" /> -->
-			<mass value="6.2229" />
-			<inertia
-				ixx="0.0001"
-				ixy="0.0001"
-				ixz="0.0001"
-				iyy="0.0001"
-				iyz="0.0001"
-				izz="0.0787" /> <!--0.00101 "-->
-		</inertial>
-		<visual>
-			<origin xyz="0.036 0 0" rpy="0 0 0"/>
-			<geometry>
-				<box size= "0.072 0.07 0.05" />
-			</geometry>
-		</visual>
-		<visual>
-			<origin
-				xyz="0.072 0 0"
-				rpy="1.5708 0 0"/>
+				rpy="0 0 0" />
+			<mass value="0.03547" />
+			<inertia
+				ixx="0.0926325136613974"
+				ixy="-0.00333421740190982"
+				ixz="0.00529966557344093"
+				iyy="0.0752633235560557"
+				iyz="0.00191940596202769"
+				izz="0.0919273463968869" />
+		</inertial>
+		<visual>
+			<origin
+				xyz="0 0 0"
+				rpy="0 0 0" />
 			<geometry>
 				<mesh filename="package://cepheus_description/urdf/meshes/left_grip.STL" />
@@ -353,7 +349,7 @@
 			<origin
 				xyz="0.0375 0 0.022"
-				rpy="1.5708 0 0" />
-			<geometry>
-				<box size="0.1082 0.07 0.05"/>
+				rpy="0 0 0" />
+			<geometry>
+				<box size="0.085 0.07 0.05"/>
 			</geometry>
 		</collision>
@@ -369,42 +365,5 @@
 		</actuator>
 	</transmission>
-	<!-- <gazebo reference="left_wrist_joint">
-		<sensor name="left_wrist_joint_force_torque" type="force_torque">
-    	<always_on>true</always_on>
-    	<update_rate>20.0</update_rate>
-    	<visualize>true</visualize>
-    	<force_torque>
-    		<frame>sensor</frame>
-    		<measure_direction>child_to_parent</measure_direction>
-    	</force_torque>
-		</sensor>
-	</gazebo> -->
-<!-- The ft_sensor plugin -->
-	<!-- <gazebo>
-		<plugin name="ft_sensor" filename="libgazebo_ros_ft_sensor.so">
-			<alwaysOn>true</alwaysOn>
-			<updateRate>10.0</updateRate>
-			<topicName>ft_sensor_topic</topicName>
-			<gaussianNoise>0.0</gaussianNoise>
-			<jointName>left_wrist_joint</jointName>
-			<visualize>true</visualize>
-		</plugin>
-	</gazebo> -->
-	<!-- <gazebo reference="left_wrist_joint">
-		<disableFixedJointLumping>true</disableFixedJointLumping>
-		<sensor name="my_cool_sensor" type="force_torque">
-			<force_torque>
-			<frame>child</frame>
-			<measure_direction>child_to_parent</measure_direction>
-			</force_torque>
-		</sensor>
-	</gazebo> -->
-	<gazebo reference="left_wrist_joint">
-		<provideFeedback>true</provideFeedback>
-		<!-- <sensor name="force_torque" type="force_torque">
-          <update_rate>30</update_rate>
-    	</sensor> -->
-	</gazebo>
-	<gazebo>
+    <gazebo>
 		<plugin name="ft_sensor" filename="libgazebo_ros_ft_sensor.so">
 			<updateRate>0</updateRate>   <!--poly shmantiko na einai 0, allios kanei bug!!!!(nikhforos)-->
@@ -418,4 +377,10 @@
 		</plugin>
 	</gazebo>
+    <gazebo reference="left_wrist_joint">
+		<provideFeedback>true</provideFeedback>
+		<!-- <sensor name="force_torque" type="force_torque">
+          <update_rate>30</update_rate>
+    	</sensor> -->
+	</gazebo>
 	<gazebo>
 		<plugin filename="libgazebo_ros_force.so" name="gazebo_ros_force" >

Commit message: eftiaksa l0, evala diagnostics()

File: src/cepheus_description/urdf/cepheus.xacro (robot description, xacro)
@@ -33,5 +33,5 @@
 				xyz="0.0 0.0 0.0"
 				rpy="0.0 0.0 0.0" />
-			<mass value="0.01" />
+			<    value="0.01" />
 			<inertia
 				ixx="1e-2"
@@ -388,5 +388,5 @@
 			<!-- <update>100</update> -->
 			<!-- <updateRate>0</updateRate> anti gia 100 -->
-			<bodyName>cepheus_base</bodyName>
+			<bodyName>left_grip</bodyName>
 			<topicName>force_base_topic</topicName>
 			<force_reference_frame>world</force_reference_frame>

Commit message: did some stuff

File: src/cepheus_description/urdf/cepheus.xacro (robot description, xacro)
@@ -33,5 +33,5 @@
 				xyz="0.0 0.0 0.0"
 				rpy="0.0 0.0 0.0" />
-			<    value="0.01" />
+			<mass value="0.01" />
 			<inertia
 				ixx="1e-2"

File: src/cepheus_description/urdf/simple_ring.xacro (robot description, xacro)
@@ -28,4 +28,5 @@
     </inertial>
   </link>
+<!--
   <link name="ring_link">
     <visual>
@@ -33,5 +34,5 @@
         <cylinder length="0.01" radius="0.1"/>
       </geometry>
-      <!-- <origin xyz="0 0 0.525" /> -->
+       //htan se sxolio afto<origin xyz="0 0 0.525" />
       <material name="blue">
         <color rgba="0 0 .8 1"/>
@@ -48,8 +49,9 @@
     </inertial>
   </link>
-  <joint name="simple_joint" type="continuous">
+-->
+  <!-- <joint name="simple_joint" type="continuous">
     <parent link="base_link"/>
     <child link="ring_link"/>
-    <!-- <origin xyz="0 0 0.5" /> -->
-  </joint>
+    //htan se sxolio afto <origin xyz="0 0 0.5" />
+  </joint> -->
 </robot>

Commit message: telos diplomatikis

File: src/cepheus_description/urdf/cepheus.xacro (robot description, xacro)
@@ -366,15 +366,4 @@
 	</transmission>
     <gazebo>
-		<plugin name="ft_sensor" filename="libgazebo_ros_ft_sensor.so">
-			<updateRate>0</updateRate>   <!--poly shmantiko na einai 0, allios kanei bug!!!!(nikhforos)-->
-			<topicName>ft_sensor_topic</topicName>
-			<jointName>left_wrist_joint</jointName>
-			<noise>
-          		<type>gaussian</type>
-          		<mean>0.0</mean>
-          		<stddev>0.003</stddev> <!-- change this to simulate noise -->
-        	</noise>
-		</plugin>
-	</gazebo>
     <gazebo reference="left_wrist_joint">
 		<provideFeedback>true</provideFeedback>

File: src/cepheus_description/urdf/cepheus_simplified.xacro (robot description, xacro)
@@ -281,5 +281,5 @@
 				rpy="0 0 0" />
 			<geometry>
-				<box size="${arm_length} 0.02 0.02" />
+				<box size="${arm_length} 0.03 0.03" />
 			</geometry>
 			<material name="LightGrey"/>
@@ -290,5 +290,5 @@
 				rpy="0 0 0" />
 			<geometry>
-				<box size="${arm_length} 0.02 0.02"/>
+				<box size="${arm_length} 0.03 0.03"/>
 			</geometry>
 		</collision>
@@ -342,5 +342,5 @@
 				rpy="0 0 0" />
 			<geometry>
-				<box size="${forearm_length} 0.02 0.02"/>
+				<box size="${forearm_length} 0.03 0.03"/>
 			</geometry>
 			<material name="LightGrey"/>
@@ -351,5 +351,5 @@
 				rpy="0 0 0" />
 			<geometry>
-				<box size="${forearm_length} 0.02 0.02"/>
+				<box size="${forearm_length} 0.03 0.03"/>
 			</geometry>
 		</collision>
@@ -403,5 +403,5 @@
 				rpy="0 0 0" />
 			<geometry>
-				<box size="${gripper_length} 0.02 0.02"/>
+				<box size="${gripper_length} 0.03 0.03"/>
 			</geometry>
 			<material name="LightGrey"/>
@@ -412,5 +412,5 @@
 				rpy="0 0 0" />
 			<geometry>
-				<box size="${gripper_length} 0.02 0.02"/>
+				<box size="${gripper_length} 0.03 0.03"/>
 			</geometry>
 			<!-- <surface>
@@ -466,5 +466,5 @@
 		<child link="final_link"/>
 		<origin
-			xyz="${gripper_length} 0 0.02"
+			xyz="${gripper_length} 0 0.03"
 			rpy="0 0 0 " />
 		<axis xyz="1 0 0"/>
@@ -513,14 +513,4 @@
           		<stddev>0.0003</stddev> <!-- change this to simulate noise -->
         	</noise>
-		</plugin>
-	</gazebo>
-	<gazebo>
-		<plugin filename="libgazebo_ros_force.so" name="gazebo_ros_force" >
-			<!-- <alwaysOn>true</alwaysOn> -->
-			<!-- <update>100</update> -->
-			<!-- <updateRate>0</updateRate> anti gia 100 -->
-			<bodyName>cepheus_base</bodyName>
-			<topicName>force_base_topic</topicName>
-			<force_reference_frame>cepheus_base</force_reference_frame>
 		</plugin>
 	</gazebo>
@@ -548,3 +538,16 @@
   </gazebo>
 	<!-- <gravity>false</gravity> -->
+	<gazebo reference="left_wrist_joint">
+		<provideFeedback>true</provideFeedback>
+	</gazebo>
+	<plugin name="ft_sensor" filename="libgazebo_ros_ft_sensor.so">
+			<updateRate>0</updateRate>   <!--poly shmantiko na einai 0, allios kanei bug!!!!(nikhforos)-->
+			<topicName>ft_sensor_topic</topicName>
+			<jointName>left_wrist_joint</jointName>
+			<noise>
+          		<type>gaussian</type>
+          		<mean>0.0</mean>
+          		<stddev>0.003</stddev> <!-- change this to simulate noise -->
+        	</noise>
+	</plugin>
 </robot>
